File: KiCad/HEC1.kicad_pcb (KiCad board)
At the start: 2 copper layers, 243.8 x 170.2 mm, 83 parts, among them J1 Barrel_Jack_Switch, J2 Conn_02x03_Odd_Even, J3 Conn_02x05_Odd_Even, J4 Conn_02x13_Odd_Even, U1 Z80CPU, U10 74LS30, U10 74LS32, U11 74LS00, U11 74LS10, U11 74LS32, U12 74LS04, U13 74LS245, U14 74LS245, U15 74LS32, U16 74LS32, U17 74LS20, U17 74LS30, U17 74LS74, U18 74LS02, U18 74LS138, U18 74LS74, U19 74LS30, U2 AS6C4008-55PCN, U20 74LS574, U21 74LS574, U22 74LS02, U23 74LS74, U24 74LS74, U25 74LS541, U26 74LS541, U27 74LS74, U28 74LS20, U29 74LS74, U3 AS6C4008-55PCN, U30 74LS74, U31 74LS32, U32 LM79M05_TO220, U33 74LS20, U34 74LS393, U35 74LS08, U36 74LS27, U4 CY7C199, U5 CY7C199, U6 74LS138, U7 28C256, U8 74LS138, U9 74LS574, X1 CXO_DIP8

Commit message: PCB Update
Some part placement, some routing, some change in schematic for easier PCB routing.
Parts:
- removed H7: MountingHole_Pad, MountingHole:MountingHole_3.2mm_M3_Pad_Via
- removed J2: Conn_02x03_Odd_Even, Connector_PinHeader_2.54mm:PinHeader_2x03_P2.54mm_Vertical
- removed the RN1 at (392.9, -50.0)
- removed the U10 at (108.3, -61.0)
- removed the U10 at (369.8, -91.8)
- removed the U10 at (325.1, 78.7)
- removed the U11 at (428.9, 50.8)
- removed the U11 at (413.7, -2.54)
- removed the U11 at (120.0, -61.0)
- removed the U12 at (191.1, -63.5)
- removed the U12 at (440.7, 50.8)
- removed the U12 at (-83.3, 66.0)
- removed the U17 at (202.9, -63.5)
- removed the U17 at (381.5, -91.8)
- removed the U17 at (325.1, -104.1)
- removed the U18 at (336.9, -104.1)
- removed the U18 at (-72.7, 30.5)
- removed the U18 at (393.3, -91.8)
- removed the U19 at (405.0, -91.8)
- removed the U19 at (348.6, -104.1)
- removed the U22 at (425.4, -2.54)
- removed the U22 at (237.0, -6.90)
- removed the U23 at (-61.0, 30.5)
- removed the U23 at (416.8, -91.8)
- removed the U24 at (428.5, -91.8)
- removed the U24 at (131.8, -61.0)
- removed the U30 at (214.6, -63.5)
- removed the U30 at (167.0, -61.0)
- removed the U6 at (413.7, 17.0)
- removed the U6 at (428.9, 72.3)
- removed the U6 at (209.6, -35.3)
- removed the U8 at (384.2, 115.6)
- removed the U8 at (96.5, -61.0)
- removed the U8 at (425.4, 17.0)
- added C10: C_Polarized, Capacitor_THT:CP_Radial_D6.3mm_P2.50mm, F.Cu at (129.5, 49.6)
- added C11: C_Polarized, Capacitor_THT:CP_Radial_D6.3mm_P2.50mm, F.Cu at (129.5, 61.2)
- added C12: C_Polarized, Capacitor_THT:CP_Radial_D10.0mm_P5.00mm, F.Cu at (92.7, 246.4)
- added C13: C, Capacitor_THT:C_Disc_D7.0mm_W2.5mm_P5.00mm, F.Cu at (102.8, 242.6)
- added C14: C, Capacitor_THT:C_Disc_D7.0mm_W2.5mm_P5.00mm, F.Cu at (102.8, 246.7)
- added C15: C, Capacitor_THT:C_Disc_D7.0mm_W2.5mm_P5.00mm, F.Cu at (102.8, 250.7)
- added C16: C, Capacitor_THT:C_Disc_D7.0mm_W2.5mm_P5.00mm, F.Cu at (102.8, 254.8)
- added C17: C, Capacitor_THT:C_Disc_D7.0mm_W2.5mm_P5.00mm, F.Cu at (102.8, 258.8)
- added C18: C, Capacitor_THT:C_Disc_D7.0mm_W2.5mm_P5.00mm, F.Cu at (102.8, 262.9)
- added C19: C, Capacitor_THT:C_Disc_D7.0mm_W2.5mm_P5.00mm, F.Cu at (111.3, 242.6)
- added C20: C, Capacitor_THT:C_Disc_D7.0mm_W2.5mm_P5.00mm, F.Cu at (111.3, 246.7)
- added C21: C_Polarized, Capacitor_THT:CP_Radial_D10.0mm_P5.00mm, F.Cu at (92.7, 257.9)
- added C22: C, Capacitor_THT:C_Disc_D7.0mm_W2.5mm_P5.00mm, F.Cu at (111.3, 250.7)
- added C23: C, Capacitor_THT:C_Disc_D7.0mm_W2.5mm_P5.00mm, F.Cu at (111.3, 254.8)
- added C24: C, Capacitor_THT:C_Disc_D7.0mm_W2.5mm_P5.00mm, F.Cu at (111.3, 258.8)
- added C25: C, Capacitor_THT:C_Disc_D7.0mm_W2.5mm_P5.00mm, F.Cu at (111.3, 262.9)
- added C26: C, Capacitor_THT:C_Disc_D7.0mm_W2.5mm_P5.00mm, F.Cu at (119.9, 242.6)
- added C27: C, Capacitor_THT:C_Disc_D7.0mm_W2.5mm_P5.00mm, F.Cu at (119.9, 246.7)
- added C28: C, Capacitor_THT:C_Disc_D7.0mm_W2.5mm_P5.00mm, F.Cu at (119.9, 250.7)
- added C29: C, Capacitor_THT:C_Disc_D7.0mm_W2.5mm_P5.00mm, F.Cu at (119.9, 254.8)
- added C30: C_Polarized, Capacitor_THT:CP_Radial_D10.0mm_P5.00mm, F.Cu at (92.7, 269.5)
- added C9: C_Polarized, Capacitor_THT:CP_Radial_D6.3mm_P2.50mm, F.Cu at (129.5, 38.1)
- added R1: R, Resistor_THT:R_Axial_DIN0207_L6.3mm_D2.5mm_P7.62mm_Horizontal, F.Cu at (343.6, 220.1)
- added RN3: R_Network04, Resistor_THT:R_Array_SIP5, F.Cu at (497.5, 67.3)
- added SW1: SW_DIP_x04, Button_Switch_THT:SW_DIP_SPSTx04_Slide_9.78x12.34mm_W7.62mm_P2.54mm, F.Cu at (63.5, 160.0)
- added SW2: SW_Push, Button_Switch_THT:SW_PUSH_6mm, F.Cu at (344.0, 224.1)
- added U10: 74LS32, Package_DIP:DIP-14_W7.62mm_Socket, F.Cu at (556.0, 53.3)
- added U10: 74LS32, Package_DIP:DIP-14_W7.62mm_Socket, F.Cu at (181.6, 135.3)
- added U11: 74LS00, Package_DIP:DIP-14_W7.62mm_Socket, F.Cu at (477.2, 104.1)
- added U12: 74LS04, Package_DIP:DIP-14_W7.62mm_Socket, F.Cu at (63.5, 138.4)
- added U17: 74LS20, Package_DIP:DIP-14_W7.62mm_Socket, F.Cu at (91.4, 130.8)
- added U18: 74LS138, Package_DIP:DIP-16_W7.62mm_Socket, F.Cu at (348.0, -10.2)
- added U19: 74LS30, Package_DIP:DIP-14_W7.62mm_Socket, F.Cu at (386.2, -73.7)
- added U22: 74LS02, Package_DIP:DIP-14_W7.62mm_Socket, F.Cu at (312.4, 44.5)
- added U23: 74LS74, Package_DIP:DIP-14_W7.62mm_Socket, F.Cu at (359.7, -10.2)
- added U24: 74LS74, Package_DIP:DIP-14_W7.62mm_Socket, F.Cu at (397.9, -73.7)
- added U30: 74LS74, Package_DIP:DIP-14_W7.62mm_Socket, F.Cu at (332.7, 74.9)
- added U37: 74LS32, Package_DIP:DIP-14_W7.62mm_Socket, F.Cu at (363.2, 109.2)
- added U6: 74LS138, Package_DIP:DIP-16_W7.62mm_Socket, F.Cu at (104.2, 128.3)
- added U8: 74LS138, Package_DIP:DIP-16_W7.62mm_Socket, F.Cu at (306.1, 87.6)
- moved U28 422.1 mm to (533.1, 101.6)
- moved U29 422.1 mm to (544.8, 101.6)
- moved U27 404.7 mm to (186.7, 223.5)
- moved U3 292.0 mm to (429.3, 167.6)
- moved U2 291.7 mm to (410.2, 167.6)
- moved U21 286.4 mm to (129.5, 71.1)
- moved U20 278.1 mm to (129.5, 99.1)
- moved C1 275.3 mm to (78.8, 236.2)
- moved C2 275.3 mm to (78.8, 241.3)
- moved C3 275.3 mm to (78.8, 246.4)
- moved C4 275.3 mm to (78.8, 251.5)
- moved C5 275.3 mm to (78.8, 256.5)
- moved C6 275.3 mm to (78.8, 261.6)
- moved C7 275.3 mm to (78.8, 266.7)
- moved C8 275.3 mm to (78.8, 271.8)
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Connections:
- BUS1 pad 18: /HEC_IO/~{IO_CS2} -> /HEC_IO/~{IO_CS4}
- BUS1 pad 19: unconnected-(BUS1-~{ROMRD}-Pad19) -> /HEC_IO/~{ROMRD}
- BUS1 pad 20: /HEC_IO/~{RD} -> /HEC_CPU/~{RD}
- BUS1 pad 27: /HEC_IO/~{RESET} -> /HEC_CPU/~{RST}
- BUS2 pad 18: /HEC_IO/~{IO_CS3} -> /HEC_IO/~{IO_CS5}
- BUS2 pad 19: unconnected-(BUS2-~{ROMRD}-Pad19) -> /HEC_IO/~{ROMRD}
- BUS2 pad 20: /HEC_IO/~{RD} -> /HEC_CPU/~{RD}
- BUS2 pad 27: /HEC_IO/~{RESET} -> /HEC_CPU/~{RST}
- BUS3 pad 18: /HEC_IO/~{IO_CS4} -> /HEC_IO/~{IO_CS6}
- BUS3 pad 19: unconnected-(BUS3-~{ROMRD}-Pad19) -> /HEC_IO/~{ROMRD}
- BUS3 pad 20: /HEC_IO/~{RD} -> /HEC_CPU/~{RD}
- BUS3 pad 27: /HEC_IO/~{RESET} -> /HEC_CPU/~{RST}
- BUS4 pad 18: Net-(BUS4-~{CS}) -> /HEC_IO/~{IO_CS7}
- BUS4 pad 19: unconnected-(BUS4-~{ROMRD}-Pad19) -> /HEC_IO/~{ROMRD}
- BUS4 pad 20: /HEC_IO/~{RD} -> /HEC_CPU/~{RD}
- BUS4 pad 27: /HEC_IO/~{RESET} -> /HEC_CPU/~{RST}
- J3 pad 1: Net-(J3-Pin_1) -> /HEC_CPU/CLK
- J3 pad 10: /HEC_CPU/CLK -> Net-(J3-Pin_10)
- J3 pad 2: /HEC_CPU/CLK -> /HEC_IO/OSC
- J3 pad 3: Net-(J3-Pin_3) -> /HEC_CPU/CLK
- J3 pad 4: /HEC_CPU/CLK -> Net-(J3-Pin_4)
- J3 pad 5: Net-(J3-Pin_5) -> /HEC_CPU/CLK
- J3 pad 6: /HEC_CPU/CLK -> Net-(J3-Pin_6)
- J3 pad 7: Net-(J3-Pin_7) -> /HEC_CPU/CLK
- J3 pad 8: /HEC_CPU/CLK -> Net-(J3-Pin_8)
- J3 pad 9: Net-(J3-Pin_9) -> /HEC_CPU/CLK
- J4 pad 1: /HEC_IO/~{IO_CS1} -> /HEC_IO/~{PSG_INT}
- J4 pad 10: /HEC_IO/D4 -> /HEC_IO/D6
- J4 pad 11: /HEC_IO/A2 -> /HEC_IO/D5
- J4 pad 12: /HEC_IO/D5 -> /HEC_IO/D4
- J4 pad 13: /HEC_IO/A3 -> /HEC_IO/D3
- J4 pad 14: /HEC_IO/D6 -> /HEC_IO/D2
- J4 pad 15: /HEC_IO/A4 -> /HEC_IO/D1
- J4 pad 16: /HEC_IO/D7 -> /HEC_IO/D0
- J4 pad 17: /HEC_IO/~{RESET} -> /HEC_IO/~{IO_CS1}
- J4 pad 18: /HEC_IO/WAIT_INTERNAL -> /HEC_CPU/~{RST}
- J4 pad 19: /HEC_IO/~{VDP_INT} -> /HEC_CPU/~{WR}
- J4 pad 2: /HEC_IO/D0 -> Net-(J4-Pin_2)
- J4 pad 20: /HEC_IO/OSC -> /HEC_IO/~{VDP_INT}
- J4 pad 21: /HEC_IO/~{PSG_INT} -> /HEC_IO/A4
- J4 pad 22: H -> /HEC_CPU/~{RD}
- J4 pad 23: /HEC_IO/~{KB_INT} -> /HEC_IO/A2
- J4 pad 24: H -> /HEC_IO/A3
- J4 pad 25: /HEC_IO/~{MS_INT} -> /HEC_IO/A0
- J4 pad 26: L -> /HEC_IO/A1
- J4 pad 3: /HEC_IO/~{RD} -> /HEC_IO/~{KB_INT}
- J4 pad 4: /HEC_IO/D1 -> /HEC_IO/~{MS_INT}
- J4 pad 5: /HEC_CPU/~{WR} -> H
- J4 pad 6: /HEC_IO/D2 -> /HEC_IO/OSC
- J4 pad 7: /HEC_IO/A0 -> H
- J4 pad 8: /HEC_IO/D3 -> L
- J4 pad 9: /HEC_IO/A1 -> /HEC_IO/D7
- RN2 pad 2: /HEC_IO/~{NOWS4} -> /HEC_IO/~{NOWS3}
- RN2 pad 3: /HEC_IO/~{NOWS3} -> /HEC_IO/~{NOWS2}
- RN2 pad 4: /HEC_IO/~{NOWS2} -> /HEC_IO/~{NOWS4}
- U1 pad 10: /HEC_Memory/D6 -> /HEC_IO/D6
- U1 pad 12: /HEC_Memory/D2 -> /HEC_IO/D2
- U1 pad 13: /HEC_Memory/D7 -> /HEC_IO/D7
- U1 pad 14: /HEC_Memory/D0 -> /HEC_IO/D0
- U1 pad 15: /HEC_Memory/D1 -> /HEC_IO/D1
- U1 pad 24: /HEC_CPU/~{CPU_WAIT} -> /HEC_CPU/~{WAIT}
- U1 pad 28: /HEC_CPU/~{RFSH} -> /MEC_Protection/~{RFSH}
- U1 pad 7: /HEC_Memory/D4 -> /HEC_IO/D4
- U1 pad 8: /HEC_Memory/D3 -> /HEC_IO/D3
- U1 pad 9: /HEC_Memory/D5 -> /HEC_IO/D5
- U13 pad 11: /HEC_Memory/RAM_A15 -> /HEC_IO/D7
- U13 pad 12: /HEC_Memory/RAM_A14 -> /HEC_IO/D6
- U13 pad 13: /HEC_Memory/RAM_A13 -> /HEC_IO/D5
- U13 pad 14: /HEC_Memory/RAM_A12 -> /HEC_IO/D4
- U13 pad 15: /HEC_Memory/RAM_A11 -> /HEC_IO/D3
- U13 pad 16: /HEC_Memory/RAM_A10 -> /HEC_IO/D2
- U13 pad 17: /HEC_Memory/RAM_A9 -> /HEC_IO/D1
- U13 pad 18: /HEC_Memory/RAM_A8 -> /HEC_IO/D0
- U13 pad 2: /HEC_Memory/D0 -> /HEC_Memory/RAM_A8
- U13 pad 3: /HEC_Memory/D1 -> /HEC_Memory/RAM_A9
- U13 pad 4: /HEC_Memory/D2 -> /HEC_Memory/RAM_A10
- U13 pad 5: /HEC_Memory/D3 -> /HEC_Memory/RAM_A11
- U13 pad 6: /HEC_Memory/D4 -> /HEC_Memory/RAM_A12
- U13 pad 7: /HEC_Memory/D5 -> /HEC_Memory/RAM_A13
- U13 pad 8: /HEC_Memory/D6 -> /HEC_Memory/RAM_A14
- U13 pad 9: /HEC_Memory/D7 -> /HEC_Memory/RAM_A15
- U14 pad 11: /HEC_Memory/ATTR_WP -> /HEC_IO/D7
- U14 pad 12: /HEC_Memory/ATTR_WI -> /HEC_IO/D6
- U14 pad 13: /HEC_Memory/ATTR_RI -> /HEC_IO/D5
- U14 pad 14: /HEC_Memory/ATTR_NX -> /HEC_IO/D4
- U14 pad 15: /HEC_Memory/RAM_A19 -> /HEC_IO/D3
- U14 pad 16: /HEC_Memory/RAM_A18 -> /HEC_IO/D2
- U14 pad 17: /HEC_Memory/RAM_A17 -> /HEC_IO/D1
- U14 pad 18: /HEC_Memory/RAM_A16 -> /HEC_IO/D0
- U14 pad 2: /HEC_Memory/D0 -> /HEC_Memory/RAM_A16
- U14 pad 3: /HEC_Memory/D1 -> /HEC_Memory/RAM_A17
- U14 pad 4: /HEC_Memory/D2 -> /HEC_Memory/RAM_A18
- U14 pad 5: /HEC_Memory/D3 -> /HEC_Memory/RAM_A19
- U14 pad 6: /HEC_Memory/D4 -> /HEC_Memory/ATTR_NX
- U14 pad 7: /HEC_Memory/D5 -> /HEC_Memory/ATTR_RI
- U14 pad 8: /HEC_Memory/D6 -> /HEC_Memory/ATTR_WI
- U14 pad 9: /HEC_Memory/D7 -> /HEC_Memory/ATTR_WP
- U15 pad 2: /HEC_Memory/WP -> /HEC_Memory/ATTR_WP
- U15 pad 4: /HEC_CPU/~{RD} -> unconnected-(U15-Pad4)
- U15 pad 5: /HEC_Memory/ROM -> unconnected-(U15-Pad5)
- U15 pad 6: /HEC_Memory/~{RAM_RD} -> unconnected-(U15-Pad6)
- U16 pad 12: /HEC_CPU/~{LATCH_H} -> /HEC_CPU/~{IOPORT_H}
- U16 pad 9: /HEC_CPU/~{LATCH_L} -> /HEC_CPU/~{IOPORT_L}
- U2 pad 13: /HEC_Memory/D0 -> /HEC_IO/D0
- U2 pad 14: /HEC_Memory/D1 -> /HEC_IO/D1
- U2 pad 15: /HEC_Memory/D2 -> /HEC_IO/D2
- U2 pad 17: /HEC_Memory/D3 -> /HEC_IO/D7
- U2 pad 18: /HEC_Memory/D4 -> /HEC_IO/D6
- U2 pad 19: /HEC_Memory/D5 -> /HEC_IO/D5
- U2 pad 20: /HEC_Memory/D6 -> /HEC_IO/D4
- U2 pad 21: /HEC_Memory/D7 -> /HEC_IO/D3
- U2 pad 24: /HEC_Memory/~{RAM_RD} -> /HEC_Memory/~{RAM_OE}
- U20 pad 12: /HEC_Memory/D7 -> /HEC_IO/D7
- U20 pad 13: /HEC_Memory/D6 -> /HEC_IO/D6
- U20 pad 14: /HEC_Memory/D5 -> /HEC_IO/D5
- U20 pad 15: /HEC_Memory/D4 -> /HEC_IO/D4
- U20 pad 16: /HEC_Memory/D3 -> /HEC_IO/D3
- U20 pad 17: /HEC_Memory/D2 -> /HEC_IO/D2
- U20 pad 18: /HEC_Memory/D1 -> /HEC_IO/D1
- U20 pad 19: /HEC_Memory/D0 -> /HEC_IO/D0
- U21 pad 12: /HEC_Memory/D7 -> /HEC_IO/D7
- U21 pad 13: /HEC_Memory/D6 -> /HEC_IO/D6
- U21 pad 14: /HEC_Memory/D5 -> /HEC_IO/D5
- U21 pad 15: /HEC_Memory/D4 -> /HEC_IO/D4
- U21 pad 16: /HEC_Memory/D3 -> /HEC_IO/D3
- U21 pad 17: /HEC_Memory/D2 -> /HEC_IO/D2
- U21 pad 18: /HEC_Memory/D1 -> /HEC_IO/D1
- U21 pad 19: /HEC_Memory/D0 -> /HEC_IO/D0
- U27 pad 9: /MEC_Protection/~{SYS} -> unconnected-(U27B-Q-Pad9)
- U3 pad 13: /HEC_Memory/D0 -> /HEC_IO/D0
- U3 pad 14: /HEC_Memory/D1 -> /HEC_IO/D1
- U3 pad 15: /HEC_Memory/D2 -> /HEC_IO/D2
- U3 pad 17: /HEC_Memory/D3 -> /HEC_IO/D7
- U3 pad 18: /HEC_Memory/D4 -> /HEC_IO/D6
- U3 pad 19: /HEC_Memory/D5 -> /HEC_IO/D5
- U3 pad 20: /HEC_Memory/D6 -> /HEC_IO/D4
- U3 pad 21: /HEC_Memory/D7 -> /HEC_IO/D3
- U3 pad 24: /HEC_Memory/~{RAM_RD} -> /HEC_Memory/~{RAM_OE}
- U31 pad 1: Net-(BUS4-~{CS}) -> /HEC_IO/~{IO_CS7}
- U31 pad 12: /HEC_IO/~{IO_CS2} -> /HEC_IO/~{IO_CS4}
- U31 pad 4: /HEC_IO/~{IO_CS4} -> /HEC_IO/~{IO_CS6}
- U31 pad 9: /HEC_IO/~{IO_CS3} -> /HEC_IO/~{IO_CS5}
- U33 pad 1: /HEC_IO/~{WAIT1} -> Net-(RN2-R5)
- U33 pad 10: Net-(RN2-R6) -> /HEC_IO/~{WAIT2}
- U33 pad 12: Net-(RN2-R7) -> /HEC_IO/~{WAIT3}
- U33 pad 13: Net-(RN2-R8) -> /HEC_IO/~{WAIT4}
- U33 pad 2: /HEC_IO/~{WAIT2} -> Net-(RN2-R6)
- U33 pad 4: /HEC_IO/~{WAIT3} -> Net-(RN2-R7)
- U33 pad 5: /HEC_IO/~{WAIT4} -> Net-(RN2-R8)
- U33 pad 6: Net-(U33-Pad6) -> Net-(U22-Pad9)
- U33 pad 8: Net-(U33-Pad8) -> Net-(U22-Pad8)
- U33 pad 9: Net-(RN2-R5) -> /HEC_IO/~{WAIT1}
- U34 pad 1: Net-(U34A-CP) -> /HEC_IO/OSC
- U34 pad 10: Net-(J3-Pin_5) -> Net-(U34B-Q1)
- U34 pad 11: Net-(J3-Pin_3) -> Net-(U34B-Q0)
- U34 pad 12: L -> Net-(U30B-Q)
- U34 pad 13: Net-(J3-Pin_1) -> Net-(U34B-CP)
- U34 pad 2: Net-(U30B-Q) -> L
- U34 pad 3: Net-(U34A-Q0) -> Net-(J3-Pin_4)
- U34 pad 4: Net-(U34A-Q1) -> Net-(J3-Pin_6)
- U34 pad 5: Net-(U34A-Q2) -> Net-(J3-Pin_8)
- U34 pad 6: Net-(U34A-Q3) -> Net-(J3-Pin_10)
- U34 pad 8: Net-(J3-Pin_9) -> Net-(U34B-Q3)
- U34 pad 9: Net-(J3-Pin_7) -> Net-(U34B-Q2)
- U35 pad 10: unconnected-(U35-Pad10) -> L
- U35 pad 12: unconnected-(U35-Pad12) -> L
- U35 pad 13: unconnected-(U35-Pad13) -> L
- U35 pad 14: unconnected-(U35E-VCC-Pad14) -> H
- U35 pad 2: Net-(U33-Pad8) -> Net-(U22-Pad9)
- U35 pad 3: Net-(U34A-CP) -> Net-(U34B-CP)
- U35 pad 4: unconnected-(U35-Pad4) -> L
- U35 pad 5: unconnected-(U35-Pad5) -> L
- U35 pad 7: unconnected-(U35E-GND-Pad7) -> L
- U35 pad 9: unconnected-(U35-Pad9) -> L
- U36 pad 10: unconnected-(U36-Pad10) -> L
- U36 pad 11: unconnected-(U36-Pad11) -> L
- U36 pad 12: /HEC_IO/~{WAIT} -> /HEC_CPU/~{WAIT}
- U36 pad 13: Net-(U33-Pad8) -> Net-(U33-Pad6)
- U36 pad 14: unconnected-(U36D-VCC-Pad14) -> H
- U36 pad 2: Net-(U33-Pad6) -> Net-(U33-Pad8)
- U36 pad 3: unconnected-(U36-Pad3) -> L
- U36 pad 4: unconnected-(U36-Pad4) -> L
- U36 pad 5: unconnected-(U36-Pad5) -> L
- U36 pad 7: unconnected-(U36D-GND-Pad7) -> L
- U36 pad 9: unconnected-(U36-Pad9) -> L
- U4 pad 20: /HEC_Memory/L -> L
- U4 pad 22: /HEC_Memory/L -> L
- U5 pad 20: /HEC_Memory/L -> L
- U5 pad 22: /HEC_Memory/L -> L
- U7 pad 11: /HEC_Memory/D0 -> /HEC_IO/D0
- U7 pad 12: /HEC_Memory/D1 -> /HEC_IO/D1
- U7 pad 13: /HEC_Memory/D2 -> /HEC_IO/D2
- U7 pad 15: /HEC_Memory/D3 -> /HEC_IO/D3
- U7 pad 16: /HEC_Memory/D4 -> /HEC_IO/D4
- U7 pad 17: /HEC_Memory/D5 -> /HEC_IO/D5
- U7 pad 18: /HEC_Memory/D6 -> /HEC_IO/D6
- U7 pad 19: /HEC_Memory/D7 -> /HEC_IO/D7
- U7 pad 22: /HEC_CPU/ROM -> /HEC_CPU/~{ROM_OE}
- U9 pad 1: /HEC_Memory/L -> L
- U9 pad 11: unconnected-(U9-Cp-Pad11) -> Net-(U9-Cp)
- U9 pad 2: /HEC_Memory/D0 -> /HEC_IO/D0
- U9 pad 3: /HEC_Memory/D1 -> /HEC_IO/D1
- U9 pad 4: /HEC_Memory/D2 -> /HEC_IO/D2
- U9 pad 5: /HEC_Memory/D3 -> /HEC_IO/D3
- U9 pad 6: /HEC_Memory/D4 -> /HEC_IO/D4
- U9 pad 7: /HEC_Memory/D5 -> /HEC_IO/D5
- U9 pad 8: /HEC_Memory/D6 -> /HEC_IO/D6
- U9 pad 9: /HEC_Memory/D7 -> /HEC_IO/D7
- X1 pad 5: Net-(J3-Pin_1) -> /HEC_IO/OSC
Routing:
- net /HEC_IO/D7: track 0.00 -> 158.0 mm
- net /HEC_IO/A0: track 0.00 -> 149.3 mm
- net /HEC_IO/A2: track 0.00 -> 149.3 mm
- net /HEC_IO/A4: track 0.00 -> 149.3 mm
- net /HEC_IO/D6: track 0.00 -> 139.7 mm
- net /HEC_IO/D5: track 0.00 -> 139.7 mm
- net /HEC_IO/A3: track 0.00 -> 131.0 mm
- net /HEC_IO/A1: track 0.00 -> 131.0 mm
- net /HEC_IO/D4: track 0.00 -> 121.4 mm
- net /HEC_IO/D3: track 0.00 -> 121.4 mm
- net /HEC_CPU/~{RD}: track 0.00 -> 119.0 mm
- net /HEC_IO/D0: track 0.00 -> 103.1 mm
- net /HEC_IO/D2: track 0.00 -> 103.1 mm
- net /HEC_IO/D1: track 0.00 -> 103.1 mm
- net /HEC_CPU/~{WR}: track 0.00 -> 100.7 mm
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
Commit message: Add POST code circuit
Add circuit to show POST code using I register on Z80 to assist debugging.
Parts:
- removed J4: Conn_02x13_Odd_Even, Connector_PinHeader_2.54mm:PinHeader_2x13_P2.54mm_Vertical
- added J2: Conn_02x12_Odd_Even, Connector_PinHeader_2.54mm:PinHeader_2x12_P2.54mm_Vertical, F.Cu at (196.2, 66.0)
- added RN3: R_Pack07, Package_DIP:DIP-14_W7.62mm, F.Cu at (102.7, -8.61)
- added RN4: R_Pack07, Package_DIP:DIP-14_W7.62mm, F.Cu at (159.4, -6.36)
- added U28: 74LS30, Package_DIP:DIP-14_W7.62mm_Socket, F.Cu at (180.3, 2.54)
- added U36: 74LS574, Package_DIP:DIP-20_W7.62mm_Socket, F.Cu at (58.7, -19.7)
- added U37: 74LS32, Package_DIP:DIP-14_W7.62mm_Socket, F.Cu at (47.0, -19.7)
- added U38: 74LS47, Package_DIP:DIP-16_W7.62mm_Socket, F.Cu at (146.7, -8.89)
- added U39: 74LS47, Package_DIP:DIP-16_W7.62mm_Socket, F.Cu at (91.4, -8.89)
- added U40: DA04-11EWA, Display_7Segment:DA04-11SURKWA, F.Cu at (120.7, -9.46)
Connections:
- net /MEC_Protection/~{RFSH} renamed /HEC_CPU/~{RFSH}

Commit message: PCB Layout attempt
Played with PCB layout a bit to get an idea of how the layout of HEC would look like. Minor updates to schematic to simplify  PCB layout.
Parts:
- removed the RN3 at (497.5, 67.3)
- removed the U10 at (556.0, 53.3)
- removed the U28 at (533.1, 101.6)
- removed the U36 at (91.4, 152.4)
- removed the U37 at (363.2, 109.2)
- added C31: C, Capacitor_THT:C_Disc_D3.4mm_W2.1mm_P2.50mm, F.Cu at (248.9, 61.0)
- added C32: C, Capacitor_THT:C_Disc_D3.4mm_W2.1mm_P2.50mm, F.Cu at (248.9, 66.0)
- added J4: Mini-DIN_6pins_ver3, Library:Connector_Mini-DIN_Female_6Pin_2rows, F.Cu at (264.5, 33.0)
- added J5: Mini-DIN_6pins_ver3, Library:Connector_Mini-DIN_Female_6Pin_2rows, F.Cu at (290.8, 11.3)
- added J6: DE9_Plug_MountingHoles, Connector_Dsub:DSUB-9_Male_Horizontal_P2.77x2.84mm_EdgePinOffset4.94mm_Housed_MountingHolesOffset7.48mm, F.Cu at (211.1, 33.3)
- added J7: AudioJack3, Connector_Audio:Jack_3.5mm_CUI_SJ1-3533NG_Horizontal, F.Cu at (252.0, 30.6)
- added J8: NES_Port_Male, Library:NES_Port_Male_Horizontal, F.Cu at (234.4, 46.4)
- added R2: R, Resistor_THT:R_Axial_DIN0207_L6.3mm_D2.5mm_P7.62mm_Horizontal, F.Cu at (419.1, 50.8)
- added RN5: R_Network07, Resistor_THT:R_Array_SIP8, F.Cu at (221.0, 50.8)
- added RN6: R_Network08, Resistor_THT:R_Array_SIP9, F.Cu at (213.6, 38.4)
- added U41: 74LS02, Package_DIP:DIP-14_W7.62mm_Socket, F.Cu at (237.5, 210.8)
- added U42: 74LS06, Package_DIP:DIP-14_W7.62mm_Socket, F.Cu at (327.7, 34.3)
- added U43: ~, Package_DIP:DIP-40_W15.24mm_Socket, F.Cu at (236.5, 56.2)
- added U44: 74LS541, Package_DIP:DIP-20_W7.62mm_Socket, F.Cu at (213.6, 43.5)
- added Y1: Crystal, Crystal:Crystal_HC18-U_Vertical, F.Cu at (241.3, 61.0)
- moved U19 391.7 mm to (114.3, 208.3)
- moved U23 280.5 mm to (204.5, 223.5)
- moved U26 276.3 mm to (129.5, 127.0)
- moved U22 251.8 mm to (91.4, 165.1)
- moved U37 195.6 mm to (163.8, 137.2)
- moved C3 185.0 mm to (106.7, 63.5), turned to 90 degrees
- moved C2 178.0 mm to (86.4, 63.5), turned to 90 degrees
- moved C1 173.2 mm to (66.0, 63.5), turned to 90 degrees
- moved U24 171.1 mm to (379.7, 96.5)
- moved U28 135.0 mm to (142.2, 132.1)
- moved U1 125.4 mm to (226.1, 87.6)
- moved U18 117.0 mm to (231.1, -15.2)
- moved U9 114.0 mm to (354.3, 149.8)
- moved RN4 83.0 mm to (83.8, -40.6)
- moved U39 63.4 mm to (38.1, -43.2)
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Connections:
- net /HEC_CPU/~{IO_CS0} renamed /HEC_IO/~{IO_CS0}
- net /MEC_Protection/~{CLRINT} renamed /HEC_Protection/~{CLRINT}
- net /MEC_Protection/~{INT_SOURCE_1} renamed /HEC_Protection/~{INT_SOURCE_1}
- net /MEC_Protection/~{INT_SOURCE_2} renamed /HEC_Protection/~{INT_SOURCE_2}
- net /MEC_Protection/~{IO_PROT} renamed /HEC_Protection/~{IO_PROT}
- net /MEC_Protection/~{M1} renamed /HEC_Protection/~{M1}
- net /MEC_Protection/~{RFAULT} renamed /HEC_Protection/~{RFAULT}
- net /MEC_Protection/~{VDP_INT} renamed /HEC_Protection/~{AUX_IRQ}
- net /MEC_Protection/~{WFAULT} renamed /HEC_Protection/~{WFAULT}
- net /MEC_Protection/~{XFAULT} renamed /HEC_Protection/~{XFAULT}
- BUS1 pad 17: H -> /HEC_IO/~{IRQ1}
- BUS1 pad 19: /HEC_IO/~{ROMRD} -> /HEC_IO/~{ROM_OE}
- BUS1 pad 20: /HEC_CPU/~{RD} -> /HEC_IO/~{IOR}
- BUS1 pad 23: unconnected-(BUS1-~{DRQ}-Pad23) -> /HEC_IO/AUDIO_L
- BUS1 pad 25: /HEC_IO/~{IRQ1} -> /HEC_IO/AUDIO_R
- BUS1 pad 27: /HEC_CPU/~{RST} -> /HEC_CPU/~{RESET}
- BUS2 pad 17: H -> /HEC_IO/~{IRQ2}
- BUS2 pad 19: /HEC_IO/~{ROMRD} -> /HEC_IO/~{ROM_OE}
- BUS2 pad 20: /HEC_CPU/~{RD} -> /HEC_IO/~{IOR}
- BUS2 pad 23: unconnected-(BUS2-~{DRQ}-Pad23) -> /HEC_IO/AUDIO_L
- BUS2 pad 25: /HEC_IO/~{IRQ2} -> /HEC_IO/AUDIO_R
- BUS2 pad 27: /HEC_CPU/~{RST} -> /HEC_CPU/~{RESET}
- BUS3 pad 17: H -> /HEC_IO/~{IRQ3}
- BUS3 pad 19: /HEC_IO/~{ROMRD} -> /HEC_IO/~{ROM_OE}
- BUS3 pad 20: /HEC_CPU/~{RD} -> /HEC_IO/~{IOR}
- BUS3 pad 23: unconnected-(BUS3-~{DRQ}-Pad23) -> /HEC_IO/AUDIO_L
- BUS3 pad 25: /HEC_IO/~{IRQ3} -> /HEC_IO/AUDIO_R
- BUS3 pad 27: /HEC_CPU/~{RST} -> /HEC_CPU/~{RESET}
- BUS4 pad 17: H -> /HEC_IO/~{IRQ4}
- BUS4 pad 19: /HEC_IO/~{ROMRD} -> /HEC_IO/~{ROM_OE}
- BUS4 pad 20: /HEC_CPU/~{RD} -> /HEC_IO/~{IOR}
- BUS4 pad 23: unconnected-(BUS4-~{DRQ}-Pad23) -> /HEC_IO/AUDIO_L
- BUS4 pad 25: /HEC_IO/~{IRQ4} -> /HEC_IO/AUDIO_R
- BUS4 pad 27: /HEC_CPU/~{RST} -> /HEC_CPU/~{RESET}
- J2 pad 10: /HEC_IO/D0 -> /HEC_Peripherals/D0
- J2 pad 12: /HEC_CPU/~{RST} -> /HEC_Peripherals/~{RESET}
- J2 pad 14: /HEC_IO/~{VDP_INT} -> /HEC_Protection/~{VDP_IRQ}
- J2 pad 23: unconnected-(J2-Pin_23-Pad23) -> /HEC_IO/AUDIO_R
- J2 pad 24: unconnected-(J2-Pin_24-Pad24) -> /HEC_IO/AUDIO_L
- J2 pad 3: /HEC_IO/D7 -> /HEC_Peripherals/D7
- J2 pad 4: /HEC_IO/D6 -> /HEC_Peripherals/D6
- J2 pad 5: /HEC_IO/D5 -> /HEC_Peripherals/D5
- J2 pad 6: /HEC_IO/D4 -> /HEC_Peripherals/D4
- J2 pad 7: /HEC_IO/D3 -> /HEC_Peripherals/D3
- J2 pad 8: /HEC_IO/D2 -> /HEC_Peripherals/D2
- J2 pad 9: /HEC_IO/D1 -> /HEC_Peripherals/D1
- R1 pad 2: /HEC_CPU/~{RST} -> /HEC_CPU/~{RESET}
- SW2 pad 1: /HEC_CPU/~{RST} -> /HEC_CPU/~{RESET}
- U1 pad 26: /HEC_CPU/~{RST} -> /HEC_CPU/~{RESET}
- U10 pad 10: /MEC_Protection/~{MREQ} -> /HEC_CPU/~{MREQ}
- U10 pad 2: Net-(U27A-~{Q}) -> Net-(U27B-~{Q})
- U10 pad 3: Net-(U27A-C) -> Net-(U27B-C)
- U10 pad 4: /MEC_Protection/ATTR_RI -> /HEC_Memory/ATTR_RI
- U10 pad 5: /MEC_Protection/~{MREQ} -> /HEC_CPU/~{MREQ}
- U10 pad 9: /MEC_Protection/ATTR_WI -> /HEC_Memory/ATTR_WI
- U11 pad 1: Net-(U27A-Q) -> Net-(U27A-D)
- U11 pad 4: Net-(U27A-Q) -> Net-(U27A-D)
- U11 pad 9: /MEC_Protection/M1 -> /HEC_Protection/M1
- U12 pad 6: /MEC_Protection/M1 -> /HEC_Protection/M1
- U15 pad 4: unconnected-(U15-Pad4) -> L
- U15 pad 5: unconnected-(U15-Pad5) -> L
- U18 pad 10: /HEC_CPU/WFAULT_H -> unconnected-(U18-O5-Pad10)
- U18 pad 11: /HEC_CPU/WFAULT_L -> unconnected-(U18-O4-Pad11)
- U18 pad 12: /HEC_CPU/RFAULT_H -> unconnected-(U18-O3-Pad12)
- U18 pad 13: /HEC_CPU/RFAULT_L -> unconnected-(U18-O2-Pad13)
- U18 pad 7: /HEC_CPU/XFAULT_H -> unconnected-(U18-O7-Pad7)
- U18 pad 9: /HEC_CPU/XFAULT_L -> unconnected-(U18-O6-Pad9)
- U19 pad 8: Net-(U27A-D) -> Net-(U27B-D)
- U22 pad 11: /MEC_Protection/SYS -> /HEC_Protection/SYS
- U22 pad 5: /MEC_Protection/SYS -> /HEC_Protection/SYS
- U23 pad 10: /HEC_CPU/~{RST} -> /HEC_CPU/~{RESET}
- U23 pad 3: /HEC_CPU/~{RFSH} -> Net-(U23A-C)
- U24 pad 12: /MEC_Protection/ATTR_NX -> /HEC_Memory/ATTR_NX
- U25 pad 3: /MEC_Protection/~{PSG_INT} -> /HEC_Protection/~{VDP_IRQ}
- U25 pad 4: /MEC_Protection/~{KB_INT} -> /HEC_Peripherals/~{KB_IRQ}
- U25 pad 5: /MEC_Protection/~{MS_INT} -> /HEC_Peripherals/~{MS_IRQ}
- U27 pad 1: /HEC_CPU/~{NMI} -> H
- U27 pad 10: H -> /HEC_Protection/~{GOUSR}
- U27 pad 11: /MEC_Protection/M1 -> Net-(U27B-C)
- U27 pad 12: Net-(U27A-Q) -> Net-(U27B-D)
- U27 pad 13: H -> /HEC_CPU/~{NMI}
- U27 pad 3: Net-(U27A-C) -> /HEC_Protection/M1
- U27 pad 4: /MEC_Protection/~{GOUSR} -> H
- U27 pad 5: Net-(U27A-Q) -> unconnected-(U27A-Q-Pad5)
- U27 pad 6: Net-(U27A-~{Q}) -> /HEC_Protection/SYS
- U27 pad 8: /MEC_Protection/SYS -> Net-(U27B-~{Q})
- U27 pad 9: unconnected-(U27B-Q-Pad9) -> Net-(U27A-D)
- U28 pad 11: /HEC_IO/~{IRQ3} -> /HEC_Peripherals/~{KB_IRQ}
- U28 pad 12: /HEC_IO/~{IRQ4} -> /HEC_Peripherals/~{MS_IRQ}
- U28 pad 2: /MEC_Protection/~{PSG_INT} -> /HEC_Protection/~{VDP_IRQ}
- U28 pad 3: /MEC_Protection/~{KB_INT} -> /HEC_IO/~{IRQ3}
- U28 pad 4: /MEC_Protection/~{MS_INT} -> /HEC_IO/~{IRQ4}
- U30 pad 2: l -> L
- U37 pad 11: unconnected-(U37-Pad11) -> /HEC_IO/~{IOR}
- U37 pad 12: unconnected-(U37-Pad12) -> /HEC_CPU/~{RD}
- U37 pad 13: unconnected-(U37-Pad13) -> /HEC_CPU/~{IORQ}
- U37 pad 3: /HEC_CPU/~{ROM_OE} -> /HEC_IO/~{ROM_OE}
- U38 pad 10: Net-(RN4-R4.2) -> Net-(RN4-R6.2)
- U38 pad 12: Net-(RN4-R6.2) -> Net-(RN4-R4.2)
- U38 pad 13: Net-(RN4-R7.2) -> Net-(RN4-R3.2)
- U38 pad 9: Net-(RN4-R3.2) -> Net-(RN4-R7.2)
- U39 pad 10: Net-(RN3-R4.2) -> Net-(RN3-R6.1)
- U39 pad 11: Net-(RN3-R5.2) -> Net-(RN3-R5.1)
- U39 pad 12: Net-(RN3-R6.2) -> Net-(RN3-R4.1)
- U39 pad 13: Net-(RN3-R7.2) -> Net-(RN3-R3.1)
- U39 pad 14: Net-(RN3-R1.2) -> Net-(RN3-R1.1)
- U39 pad 15: Net-(RN3-R2.2) -> Net-(RN3-R2.1)
- U39 pad 9: Net-(RN3-R3.2) -> Net-(RN3-R7.1)
- U40 pad 1: Net-(RN3-R5.1) -> Net-(RN3-R5.2)
- U40 pad 10: Net-(RN4-R7.1) -> Net-(RN4-R3.1)
- U40 pad 12: Net-(RN4-R6.1) -> Net-(RN4-R4.1)
- U40 pad 13: Net-(RN3-R6.1) -> Net-(RN3-R4.2)
- U40 pad 14: Net-(RN3-R2.1) -> Net-(RN3-R2.2)
- U40 pad 15: Net-(RN3-R7.1) -> Net-(RN3-R3.2)
- U40 pad 16: Net-(RN3-R1.1) -> Net-(RN3-R1.2)
- U40 pad 2: Net-(RN3-R3.1) -> Net-(RN3-R7.2)
- U40 pad 3: Net-(RN3-R4.1) -> Net-(RN3-R6.2)
- U40 pad 6: Net-(RN4-R4.1) -> Net-(RN4-R6.1)
- U40 pad 7: Net-(RN4-R3.1) -> Net-(RN4-R7.1)
- U6 pad 6: /MEC_Protection/SYS -> /HEC_Protection/SYS
- U7 pad 22: /HEC_CPU/~{ROM_OE} -> /HEC_IO/~{ROM_OE}
- U8 pad 7: /MEC_Protection/~{GOUSR} -> /HEC_Protection/~{GOUSR}
Routing:
- net /HEC_IO/~{IOR}: track 0.00 -> 119.0 mm
- net /HEC_CPU/~{RD}: track 119.0 -> 0.00 mm
- net /HEC_CPU/~{RST}: track 64.1 -> 0.00 mm
- net /HEC_CPU/~{RESET}: track 0.00 -> 64.1 mm
- net /HEC_IO/~{ROM_OE}: track 0.00 -> 64.1 mm
- net /HEC_IO/~{ROMRD}: track 64.1 -> 0.00 mm

Commit message: double Mini DIN 6 port
Added double Mini DIN 6 port to replace two Mini DIN 6 port to save cost and simplify building process. The footprint is derived from the existing single mini DIN 6 port. With changes according to the png schematic. This is my first attempt at creating a footprint beyond simple 0.1inch pads, so it may be wrong. Minor changes to the PCB.
Parts:
- moved U39 427.1 mm to (421.6, 144.8)
- moved U40 427.1 mm to (445.8, 161.2)
- moved RN4 427.1 mm to (467.4, 147.3)
- moved U36 427.1 mm to (408.9, 139.7)
- moved U38 427.1 mm to (480.1, 144.8)
- moved RN3 427.1 mm to (434.3, 147.3)
- moved U29 348.0 mm to (203.2, 167.6)
- moved U11 310.5 mm to (172.7, 165.1)
- moved U25 297.3 mm to (132.1, 160.0)
- moved U24 206.1 mm to (185.4, 165.1)
- moved U8 162.4 mm to (144.8, 106.7)
- moved U18 140.5 mm to (161.3, 106.7)
- moved U1 131.4 mm to (340.4, 152.4)
- moved R1 125.4 mm to (218.4, 228.6)
- moved SW2 125.4 mm to (218.9, 232.7)
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
Commit message: Preliminary layout
Very early stage layout prototype, very subject to change.
Parts:
- removed J5: Mini-DIN_6pins_ver3, Library:Connector_Mini-DIN_Female_6Pin_2rows
- added C33: C_Polarized, Capacitor_THT:CP_Radial_D10.0mm_P5.00mm, F.Cu at (43.2, 60.9)
- added C34: C_Polarized, Capacitor_THT:CP_Radial_D10.0mm_P5.00mm, F.Cu at (5.08, 46.9)
- added C35: C_Polarized, Capacitor_THT:CP_Radial_D10.0mm_P5.00mm, F.Cu at (5.08, 58.4)
- added H10: MountingHole, MountingHole:MountingHole_3.2mm_M3, F.Cu at (242.8, 77.2)
- added H7: MountingHole, MountingHole:MountingHole_3.2mm_M3, F.Cu at (153.3, 55.7)
- added H8: MountingHole, MountingHole:MountingHole_3.2mm_M3, F.Cu at (242.8, 45.7)
- added H9: MountingHole, MountingHole:MountingHole_3.2mm_M3, F.Cu at (153.3, 77.2)
- J4: value Mini-DIN_6pins_ver3 -> ~; footprint Library:Connector_Mini-DIN_Female_6Pin_2rows -> Library:Connector_double_mini-DIN_6
- moved R2 313.4 mm to (124.5, 157.5), turned to -90 degrees
- moved U40 304.9 mm to (147.3, 99.1)
- moved RN4 303.9 mm to (175.3, 63.5)
- moved U38 303.9 mm to (188.0, 61.0)
- moved U39 293.5 mm to (152.4, 27.9)
- moved RN3 293.5 mm to (165.1, 30.5)
- moved U36 260.2 mm to (162.6, 55.9)
- moved C4 259.0 mm to (236.2, 45.7), turned to -90 degrees
- moved U30 259.0 mm to (94.0, 175.3)
- moved C30 231.4 mm to (175.3, 53.3)
- moved U3 176.4 mm to (259.1, 116.8)
- moved U2 176.4 mm to (240.0, 116.8)
- moved U13 172.7 mm to (214.6, 132.1)
- moved U14 172.7 mm to (227.3, 132.1)
- moved U4 172.7 mm to (214.6, 94.0)
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Connections:
- RN1 pad 2: /HEC_IO/~{IRQ4} -> /HEC_IO/~{SENSE1}
- RN1 pad 3: /HEC_IO/~{IRQ3} -> /HEC_IO/~{SENSE2}
- RN1 pad 4: /HEC_IO/~{IRQ2} -> /HEC_IO/~{SENSE3}
- RN1 pad 5: /HEC_IO/~{IRQ1} -> /HEC_IO/~{SENSE4}
- RN1 pad 6: /HEC_IO/~{SENSE4} -> /HEC_IO/~{IRQ1}
- RN1 pad 7: /HEC_IO/~{SENSE3} -> /HEC_IO/~{IRQ2}
- RN1 pad 8: /HEC_IO/~{SENSE2} -> /HEC_IO/~{IRQ3}
- RN1 pad 9: /HEC_IO/~{SENSE1} -> /HEC_IO/~{IRQ4}
- U10 pad 11: Net-(U9-Cp) -> unconnected-(U10-Pad11)
- U10 pad 12: /HEC_Memory/~{PID} -> L
- U10 pad 13: /HEC_CPU/~{WR} -> L
- U15 pad 4: L -> /HEC_Memory/~{PID}
- U15 pad 5: L -> /HEC_CPU/~{WR}
- U15 pad 6: unconnected-(U15-Pad6) -> Net-(U9-Cp)
- U42 pad 10: /HEC_Peripherals/~{KB_IRQ} -> Net-(RN5-R4)
- U42 pad 11: Net-(U43-KB_OBFO) -> Net-(U43-KBDO)
- U42 pad 12: /HEC_Peripherals/~{MS_IRQ} -> Net-(RN5-R5)
- U42 pad 13: Net-(U43-MS_OBFO) -> Net-(U43-KBCO)
- U42 pad 5: Net-(U43-KBDO) -> Net-(U43-KB_OBFO)
- U42 pad 6: Net-(RN5-R4) -> /HEC_Peripherals/~{KB_IRQ}
- U42 pad 8: Net-(RN5-R5) -> /HEC_Peripherals/~{MS_IRQ}
- U42 pad 9: Net-(U43-KBCO) -> Net-(U43-MS_OBFO)
Routing:
- net /HEC_IO/AUDIO_R: track 0.00 -> 64.1 mm
- net /HEC_IO/AUDIO_L: track 0.00 -> 64.1 mm
- net /HEC_IO/~{SENSE4}: track 0.00 -> 5.08 mm
- net /HEC_IO/~{SENSE3}: track 0.00 -> 5.08 mm
- net /HEC_IO/~{SENSE2}: track 0.00 -> 5.08 mm
- net /HEC_IO/~{SENSE1}: track 0.00 -> 5.08 mm
- net /HEC_IO/~{IRQ4}: track 0.00 -> 5.08 mm
- net /HEC_IO/~{IRQ3}: track 0.00 -> 5.08 mm
- net /HEC_IO/~{IRQ2}: track 0.00 -> 5.08 mm
- net /HEC_IO/~{IRQ1}: track 0.00 -> 5.08 mm
- net /HEC_IO/A4: track 149.3 -> 150.3 mm
- net /HEC_IO/A1: track 131.0 -> 132.0 mm
- net /HEC_IO/A0: track 149.3 -> 150.3 mm
- net /HEC_IO/A3: track 131.0 -> 132.0 mm
- net /HEC_IO/A2: track 149.3 -> 150.3 mm
