File: KiCad/HEC1.kicad_pcb (KiCad board)
At the start: 2 copper layers, 243.8 x 170.2 mm, 113 parts, among them J1 Barrel_Jack_Switch, J2 Conn_02x12_Odd_Even, J3 Conn_02x05_Odd_Even, J6 DE9_Plug_MountingHoles, J7 AudioJack3, J8 NES_Port_Male, SW1 SW_DIP_x04, SW2 SW_Push, U1 Z80CPU, U10 74LS32, U11 74LS00, U12 74LS04, U13 74LS245, U14 74LS245, U15 74LS32, U16 74LS32, U17 74LS20, U18 74LS138, U19 74LS30, U2 AS6C4008-55PCN, U20 74LS574, U21 74LS574, U22 74LS02, U23 74LS74, U24 74LS74, U25 74LS541, U26 74LS541, U27 74LS74, U28 74LS30, U29 74LS74, U3 AS6C4008-55PCN, U30 74LS74, U31 74LS32, U32 LM79M05_TO220, U33 74LS20, U34 74LS393, U35 74LS08, U36 74LS574, U37 74LS32, U38 74LS47, U39 74LS47, U4 CY7C199, U40 DA04-11EWA, U41 74LS02, U42 74LS06, U44 74LS541, U5 CY7C199, U6 74LS138, U7 28C256, U8 74LS138, U9 74LS574, X1 CXO_DIP8, Y1 Crystal

Commit message: Updated layout
Updated the layout of PCB. Chips on the board in this version might be in their final position.
Parts:
- added J5: Screw_Terminal_01x02, TerminalBlock_MetzConnect:TerminalBlock_MetzConnect_Type073_RT02602HBLU_1x02_P5.08mm_Horizontal, F.Cu at (271.8, 88.9)
- moved U40 288.9 mm to (426.7, 25.4)
- moved C34 257.4 mm to (259.1, 88.8), turned to 90 degrees
- moved RN4 255.8 mm to (429.3, 33.0)
- moved RN3 249.6 mm to (414.0, 12.7)
- moved U39 249.6 mm to (401.3, 10.2)
- moved U38 241.4 mm to (429.3, 53.3)
- moved U36 231.7 mm to (388.6, 5.08)
- moved U15 197.3 mm to (304.8, -63.5)
- moved U4 173.2 mm to (363.2, 5.08)
- moved U5 173.2 mm to (375.9, 5.08)
- moved U1 172.5 mm to (341.6, 19.1)
- moved U7 172.5 mm to (320.0, 20.3)
- moved U14 171.9 mm to (375.9, 45.7)
- moved U13 171.9 mm to (363.2, 45.7)
- moved U3 170.6 mm to (407.7, 33.0)
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Connections:
- U10 pad 4: /HEC_Memory/ATTR_RI -> unconnected-(U10-Pad4)
- U22 pad 13: Net-(U30A-C) -> Net-(U23B-C)
- U23 pad 10: /HEC_CPU/~{RESET} -> /HEC_Protection/~{CLRINT}
- U23 pad 11: L -> Net-(U23B-C)
- U23 pad 13: /HEC_CPU/~{RAMEN} -> H
- U23 pad 8: Net-(U23B-~{Q}) -> unconnected-(U23B-~{Q}-Pad8)
- U23 pad 9: Net-(U23B-Q) -> /HEC_Protection/~{IO_PROT}
- U30 pad 1: H -> /HEC_CPU/~{RAMEN}
- U30 pad 3: Net-(U30A-C) -> L
- U30 pad 4: /HEC_Protection/~{CLRINT} -> /HEC_CPU/~{RESET}
- U30 pad 5: /HEC_Protection/~{IO_PROT} -> Net-(U30A-Q)
- U30 pad 6: unconnected-(U30A-~{Q}-Pad6) -> Net-(U30A-~{Q})
- U37 pad 1: Net-(U23B-~{Q}) -> Net-(U30A-~{Q})
- U37 pad 11: /HEC_IO/~{IOR} -> unconnected-(U37-Pad11)
- U37 pad 12: /HEC_CPU/~{RD} -> L
- U37 pad 13: /HEC_CPU/~{IORQ} -> L
- U37 pad 4: Net-(U23B-Q) -> Net-(U30A-Q)
- U6 pad 5: /HEC_CPU/~{IORQ} -> /HEC_IO/~{IORQ}

Commit message: New bus symbol
Updated bus symbol and footprint to simplify PCB layout.
Parts:
- added R3: R, Resistor_THT:R_Axial_DIN0207_L6.3mm_D2.5mm_P7.62mm_Horizontal, F.Cu at (45.7, 88.9)
- moved U9 167.7 mm to (345.4, -17.8)
- moved C7 147.5 mm to (106.7, 121.8), turned to 90 degrees
- moved C6 139.9 mm to (86.4, 121.9), turned to 90 degrees
- moved C5 135.2 mm to (66.0, 121.9), turned to 90 degrees
- moved U17 22.9 mm to (94.0, 152.4)
- moved U22 22.9 mm to (94.0, 129.5)
- moved U40 15.2 mm to (426.7, 10.2), turned to 0 degrees
Connections:
- BUS1 pad 17: /HEC_IO/~{IRQ1} -> /HEC_IO/~{ROM_OE}
- BUS1 pad 18: /HEC_IO/~{IO_CS4} -> /HEC_IO/~{IOR}
- BUS1 pad 19: /HEC_IO/~{ROM_OE} -> /HEC_IO/~{ROM_WE}
- BUS1 pad 20: /HEC_IO/~{IOR} -> /HEC_CPU/~{WR}
- BUS1 pad 21: H -> /HEC_IO/AUDIO_L
- BUS1 pad 22: /HEC_CPU/~{WR} -> /HEC_IO/A0
- BUS1 pad 23: /HEC_IO/AUDIO_L -> /HEC_IO/AUDIO_R
- BUS1 pad 24: /HEC_IO/A0 -> /HEC_IO/A1
- BUS1 pad 25: /HEC_IO/AUDIO_R -> /HEC_CPU/~{RESET}
- BUS1 pad 26: /HEC_IO/A1 -> /HEC_IO/A2
- BUS1 pad 27: /HEC_CPU/~{RESET} -> /HEC_IO/OSC
- BUS1 pad 28: /HEC_IO/A2 -> /HEC_IO/A3
- BUS1 pad 29: /HEC_IO/OSC -> /HEC_IO/~{WAIT1}
- BUS1 pad 30: /HEC_IO/A3 -> /HEC_IO/A4
- BUS1 pad 31: /HEC_IO/~{WAIT1} -> /HEC_IO/~{IRQ1}
- BUS1 pad 32: /HEC_IO/A4 -> /HEC_IO/~{IO_CS4}
- BUS2 pad 17: /HEC_IO/~{IRQ2} -> /HEC_IO/~{ROM_OE}
- BUS2 pad 18: /HEC_IO/~{IO_CS5} -> /HEC_IO/~{IOR}
- BUS2 pad 19: /HEC_IO/~{ROM_OE} -> /HEC_IO/~{ROM_WE}
- BUS2 pad 20: /HEC_IO/~{IOR} -> /HEC_CPU/~{WR}
- BUS2 pad 21: H -> /HEC_IO/AUDIO_L
- BUS2 pad 22: /HEC_CPU/~{WR} -> /HEC_IO/A0
- BUS2 pad 23: /HEC_IO/AUDIO_L -> /HEC_IO/AUDIO_R
- BUS2 pad 24: /HEC_IO/A0 -> /HEC_IO/A1
- BUS2 pad 25: /HEC_IO/AUDIO_R -> /HEC_CPU/~{RESET}
- BUS2 pad 26: /HEC_IO/A1 -> /HEC_IO/A2
- BUS2 pad 27: /HEC_CPU/~{RESET} -> /HEC_IO/OSC
- BUS2 pad 28: /HEC_IO/A2 -> /HEC_IO/A3
- BUS2 pad 29: /HEC_IO/OSC -> /HEC_IO/~{WAIT2}
- BUS2 pad 30: /HEC_IO/A3 -> /HEC_IO/A4
- BUS2 pad 31: /HEC_IO/~{WAIT2} -> /HEC_IO/~{IRQ2}
- BUS2 pad 32: /HEC_IO/A4 -> /HEC_IO/~{IO_CS5}
- BUS3 pad 17: /HEC_IO/~{IRQ3} -> /HEC_IO/~{ROM_OE}
- BUS3 pad 18: /HEC_IO/~{IO_CS6} -> /HEC_IO/~{IOR}
- BUS3 pad 19: /HEC_IO/~{ROM_OE} -> /HEC_IO/~{ROM_WE}
- BUS3 pad 20: /HEC_IO/~{IOR} -> /HEC_CPU/~{WR}
- BUS3 pad 21: H -> /HEC_IO/AUDIO_L
- BUS3 pad 22: /HEC_CPU/~{WR} -> /HEC_IO/A0
- BUS3 pad 23: /HEC_IO/AUDIO_L -> /HEC_IO/AUDIO_R
- BUS3 pad 24: /HEC_IO/A0 -> /HEC_IO/A1
- BUS3 pad 25: /HEC_IO/AUDIO_R -> /HEC_CPU/~{RESET}
- BUS3 pad 26: /HEC_IO/A1 -> /HEC_IO/A2
- BUS3 pad 27: /HEC_CPU/~{RESET} -> /HEC_IO/OSC
- BUS3 pad 28: /HEC_IO/A2 -> /HEC_IO/A3
- BUS3 pad 29: /HEC_IO/OSC -> /HEC_IO/~{WAIT3}
- BUS3 pad 30: /HEC_IO/A3 -> /HEC_IO/A4
- BUS3 pad 31: /HEC_IO/~{WAIT3} -> /HEC_IO/~{IRQ3}
- BUS3 pad 32: /HEC_IO/A4 -> /HEC_IO/~{IO_CS6}
- BUS4 pad 17: /HEC_IO/~{IRQ4} -> /HEC_IO/~{ROM_OE}
- BUS4 pad 18: /HEC_IO/~{IO_CS7} -> /HEC_IO/~{IOR}
- BUS4 pad 19: /HEC_IO/~{ROM_OE} -> /HEC_IO/~{ROM_WE}
- BUS4 pad 20: /HEC_IO/~{IOR} -> /HEC_CPU/~{WR}
- BUS4 pad 21: H -> /HEC_IO/AUDIO_L
- BUS4 pad 22: /HEC_CPU/~{WR} -> /HEC_IO/A0
- BUS4 pad 23: /HEC_IO/AUDIO_L -> /HEC_IO/AUDIO_R
- BUS4 pad 24: /HEC_IO/A0 -> /HEC_IO/A1
- BUS4 pad 25: /HEC_IO/AUDIO_R -> /HEC_CPU/~{RESET}
- BUS4 pad 26: /HEC_IO/A1 -> /HEC_IO/A2
- BUS4 pad 27: /HEC_CPU/~{RESET} -> /HEC_IO/OSC
- BUS4 pad 28: /HEC_IO/A2 -> /HEC_IO/A3
- BUS4 pad 29: /HEC_IO/OSC -> /HEC_IO/~{WAIT4}
- BUS4 pad 30: /HEC_IO/A3 -> /HEC_IO/A4
- BUS4 pad 31: /HEC_IO/~{WAIT4} -> /HEC_IO/~{IRQ4}
- BUS4 pad 32: /HEC_IO/A4 -> /HEC_IO/~{IO_CS7}
- U19 pad 1: /HEC_IO/D0 -> /HEC_IO/D6
- U19 pad 12: H -> /HEC_Memory/SYSGATE
- U19 pad 2: /HEC_IO/D1 -> /HEC_IO/D7
- U19 pad 3: /HEC_IO/D2 -> H
- U19 pad 4: /HEC_IO/D6 -> /HEC_IO/D0
- U19 pad 5: /HEC_IO/D7 -> /HEC_IO/D1
- U19 pad 6: /HEC_Memory/SYSGATE -> /HEC_IO/D2
- U28 pad 1: /HEC_Protection/~{AUX_IRQ} -> /HEC_IO/~{IRQ1}
- U28 pad 11: /HEC_Peripherals/~{KB_IRQ} -> /HEC_IO/~{IRQ4}
- U28 pad 12: /HEC_Peripherals/~{MS_IRQ} -> /HEC_IO/~{IRQ3}
- U28 pad 2: /HEC_Protection/~{VDP_IRQ} -> /HEC_IO/~{IRQ2}
- U28 pad 3: /HEC_IO/~{IRQ3} -> /HEC_Protection/~{AUX_IRQ}
- U28 pad 4: /HEC_IO/~{IRQ4} -> /HEC_Protection/~{VDP_IRQ}
- U28 pad 5: /HEC_IO/~{IRQ1} -> /HEC_Peripherals/~{KB_IRQ}
- U28 pad 6: /HEC_IO/~{IRQ2} -> /HEC_Peripherals/~{MS_IRQ}
Routing:
- net L: track 0.00 -> 203.2 mm
- net H: track 0.00 -> 132.1 mm
- net /HEC_IO/~{ROM_WE}: track 0.00 -> 64.1 mm
- net /HEC_IO/A1: track 132.0 -> 151.4 mm
- net /HEC_IO/A3: track 132.0 -> 151.4 mm
- net /HEC_CPU/~{WR}: track 100.7 -> 119.0 mm
- net /HEC_IO/A0: track 150.3 -> 133.1 mm
- net /HEC_IO/A4: track 150.3 -> 133.1 mm
- net /HEC_IO/A2: track 150.3 -> 133.1 mm

Commit message: Exchange RI and NX pins on bus driver
A mistake is found in the schematic: the RI and NX bits are exchanged on the 74245 bus driver chip. The mistake has been corrected. This change is significant since it changes the (non-existent) software programming model. More playing around with the layout.
Parts:
- added RN7: R_Network04, Resistor_THT:R_Array_SIP5, F.Cu at (74.9, 152.4)
- RN2: value R_Network08 -> R_Network04; footprint Resistor_THT:R_Array_SIP9 -> Resistor_THT:R_Array_SIP5
- moved C34 219.3 mm to (472.4, 139.6)
- moved J5 219.3 mm to (485.1, 139.7)
- moved C35 208.6 mm to (62.2, 259.1)
- moved U15 190.9 mm to (223.5, 109.2)
- moved U16 190.9 mm to (223.5, 134.6)
- moved U37 110.3 mm to (200.7, 109.2)
- moved C12 72.3 mm to (78.7, 248.9)
- moved R1 32.5 mm to (63.5, 180.3)
- moved SW2 32.5 mm to (64.0, 184.4)
- moved X1 31.1 mm to (38.1, 114.3)
- moved U18 27.5 mm to (144.8, 83.8)
- moved SW1 25.4 mm to (63.5, 134.6)
- moved J3 22.9 mm to (43.2, 132.1)
- moved U31 22.9 mm to (78.7, 152.4)
- moved U33 22.9 mm to (78.7, 129.5)
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Connections:
- RN2 pad 2: /HEC_IO/~{NOWS3} -> Net-(RN2-R1)
- RN2 pad 3: /HEC_IO/~{NOWS2} -> Net-(RN2-R2)
- RN2 pad 4: /HEC_IO/~{NOWS4} -> Net-(RN2-R3)
- RN2 pad 5: /HEC_IO/~{NOWS1} -> Net-(RN2-R4)
- SW1 pad 5: Net-(RN2-R8) -> Net-(RN2-R4)
- SW1 pad 6: Net-(RN2-R7) -> Net-(RN2-R3)
- SW1 pad 7: Net-(RN2-R6) -> Net-(RN2-R2)
- SW1 pad 8: Net-(RN2-R5) -> Net-(RN2-R1)
- U14 pad 6: /HEC_Memory/ATTR_NX -> /HEC_Memory/ATTR_RI
- U14 pad 7: /HEC_Memory/ATTR_RI -> /HEC_Memory/ATTR_NX
- U33 pad 1: Net-(RN2-R5) -> Net-(RN2-R1)
- U33 pad 2: Net-(RN2-R6) -> Net-(RN2-R2)
- U33 pad 4: Net-(RN2-R7) -> Net-(RN2-R3)
- U33 pad 5: Net-(RN2-R8) -> Net-(RN2-R4)
- U36 pad 2: /HEC_IO/A8 -> /HEC_IO/A9
- U36 pad 3: /HEC_IO/A9 -> /HEC_IO/A10
- U36 pad 4: /HEC_IO/A10 -> /HEC_IO/A8
- U39 pad 1: Net-(U36-Q1) -> Net-(U36-Q0)
- U39 pad 14: Net-(RN3-R1.1) -> Net-(RN3-R2.1)
- U39 pad 15: Net-(RN3-R2.1) -> Net-(RN3-R1.1)
- U39 pad 2: Net-(U36-Q2) -> Net-(U36-Q1)
- U39 pad 7: Net-(U36-Q0) -> Net-(U36-Q2)
- U4 pad 1: /HEC_IO/A13 -> /HEC_Memory/PROC_ID0
- U4 pad 10: /HEC_Memory/PROC_ID6 -> /HEC_IO/A15
- U4 pad 2: /HEC_IO/A14 -> /HEC_Memory/PROC_ID1
- U4 pad 25: /HEC_IO/A11 -> /HEC_Memory/PROC_ID5
- U4 pad 26: /HEC_IO/A12 -> /HEC_Memory/PROC_ID6
- U4 pad 3: /HEC_IO/A15 -> /HEC_Memory/PROC_ID2
- U4 pad 4: /HEC_Memory/PROC_ID0 -> /HEC_Memory/PROC_ID3
- U4 pad 5: /HEC_Memory/PROC_ID1 -> /HEC_Memory/PROC_ID4
- U4 pad 6: /HEC_Memory/PROC_ID2 -> /HEC_IO/A11
- U4 pad 7: /HEC_Memory/PROC_ID3 -> /HEC_IO/A12
- U4 pad 8: /HEC_Memory/PROC_ID4 -> /HEC_IO/A13
- U4 pad 9: /HEC_Memory/PROC_ID5 -> /HEC_IO/A14
- U40 pad 14: Net-(RN3-R2.2) -> Net-(RN3-R1.2)
- U40 pad 16: Net-(RN3-R1.2) -> Net-(RN3-R2.2)
- U5 pad 1: /HEC_IO/A13 -> /HEC_Memory/PROC_ID0
- U5 pad 10: /HEC_Memory/PROC_ID6 -> /HEC_IO/A15
- U5 pad 2: /HEC_IO/A14 -> /HEC_Memory/PROC_ID1
- U5 pad 25: /HEC_IO/A11 -> /HEC_Memory/PROC_ID5
- U5 pad 26: /HEC_IO/A12 -> /HEC_Memory/PROC_ID6
- U5 pad 3: /HEC_IO/A15 -> /HEC_Memory/PROC_ID2
- U5 pad 4: /HEC_Memory/PROC_ID0 -> /HEC_Memory/PROC_ID3
- U5 pad 5: /HEC_Memory/PROC_ID1 -> /HEC_Memory/PROC_ID4
- U5 pad 6: /HEC_Memory/PROC_ID2 -> /HEC_IO/A11
- U5 pad 7: /HEC_Memory/PROC_ID3 -> /HEC_IO/A12
- U5 pad 8: /HEC_Memory/PROC_ID4 -> /HEC_IO/A13
- U5 pad 9: /HEC_Memory/PROC_ID5 -> /HEC_IO/A14
Routing:
- net /HEC_IO/OSC: track 84.7 -> 64.1 mm
- net /HEC_IO/~{NOWS4}: track 15.1 -> 0.00 mm
- net Net-(RN2-R6): track 11.5 -> 0.00 mm
- net Net-(RN2-R5): track 11.5 -> 0.00 mm
- net /HEC_CPU/CLK: track 10.2 -> 0.00 mm
- net Net-(RN2-R7): track 9.71 -> 0.00 mm
- net Net-(RN2-R8): track 9.71 -> 0.00 mm
- net /HEC_IO/~{NOWS3}: track 7.93 -> 0.00 mm
- net /HEC_IO/~{NOWS2}: track 5.39 -> 0.00 mm
- net /HEC_IO/~{NOWS1}: track 5.39 -> 0.00 mm
- net Net-(U34B-Q3): track 5.08 -> 0.00 mm
- net Net-(U34B-Q2): track 5.08 -> 0.00 mm
- net Net-(U34B-Q1): track 5.08 -> 0.00 mm
- net Net-(U34B-Q0): track 5.08 -> 0.00 mm
- net Net-(J3-Pin_8): track 3.81 -> 0.00 mm
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
Commit message: Add prototyping region
Add some prototyping regions to the board, since there WILL be bugs!
Parts:
- added J9: Conn_02x14_Odd_Even, Connector_PinHeader_2.54mm:PinHeader_2x14_P2.54mm_Vertical, F.Cu at (160.0, 83.8)
- added REF**: A_Single_Pad, Library:A_Single_Pad, F.Cu at (172.7, 58.4)
- added REF**: A_Single_Pad, Library:A_Single_Pad, F.Cu at (238.8, 185.4)
- added REF**: A_Single_Pad, Library:A_Single_Pad, F.Cu at (53.3, 165.1)
- added REF**: A_Single_Pad, Library:A_Single_Pad, F.Cu at (180.3, 58.4)
- added REF**: A_Single_Pad, Library:A_Single_Pad, F.Cu at (45.7, 162.6)
- added REF**: A_Single_Pad, Library:A_Single_Pad, F.Cu at (38.1, 180.3)
- added REF**: A_Single_Pad, Library:A_Single_Pad, F.Cu at (58.4, 180.3)
- added REF**: A_Single_Pad, Library:A_Single_Pad, F.Cu at (256.5, 180.3)
- added REF**: A_Single_Pad, Library:A_Single_Pad, F.Cu at (175.3, 61.0)
- added REF**: A_Single_Pad, Library:A_Single_Pad, F.Cu at (53.3, 167.6)
- added REF**: A_Single_Pad, Library:A_Single_Pad, F.Cu at (48.3, 172.7)
- added REF**: A_Single_Pad, Library:A_Single_Pad, F.Cu at (48.3, 175.3)
- added REF**: A_Single_Pad, Library:A_Single_Pad, F.Cu at (259.1, 170.2)
- added REF**: A_Single_Pad, Library:A_Single_Pad, F.Cu at (162.6, 55.9)
- added REF**: A_Single_Pad, Library:A_Single_Pad, F.Cu at (58.4, 167.6)
- added REF**: A_Single_Pad, Library:A_Single_Pad, F.Cu at (251.5, 172.7)
- added REF**: A_Single_Pad, Library:A_Single_Pad, F.Cu at (172.7, 53.3)
- added REF**: A_Single_Pad, Library:A_Single_Pad, F.Cu at (243.8, 165.1)
- added REF**: A_Single_Pad, Library:A_Single_Pad, F.Cu at (215.9, 193.0)
- added REF**: A_Single_Pad, Library:A_Single_Pad, F.Cu at (170.2, 73.7)
- added REF**: A_Single_Pad, Library:A_Single_Pad, F.Cu at (223.5, 185.4)
- added REF**: A_Single_Pad, Library:A_Single_Pad, F.Cu at (162.6, 66.0)
- added REF**: A_Single_Pad, Library:A_Single_Pad, F.Cu at (259.1, 172.7)
- added REF**: A_Single_Pad, Library:A_Single_Pad, F.Cu at (167.6, 50.8)
- added REF**: A_Single_Pad, Library:A_Single_Pad, F.Cu at (221.0, 182.9)
- added REF**: A_Single_Pad, Library:A_Single_Pad, F.Cu at (38.1, 157.5)
- added REF**: A_Single_Pad, Library:A_Single_Pad, F.Cu at (261.6, 175.3)
- added REF**: A_Single_Pad, Library:A_Single_Pad, F.Cu at (160.0, 66.0)
- added REF**: A_Single_Pad, Library:A_Single_Pad, F.Cu at (238.8, 172.7)
- added REF**: A_Single_Pad, Library:A_Single_Pad, F.Cu at (238.8, 165.1)
- added REF**: A_Single_Pad, Library:A_Single_Pad, F.Cu at (185.4, 63.5)
- added REF**: A_Single_Pad, Library:A_Single_Pad, F.Cu at (190.5, 185.4)
- added REF**: A_Single_Pad, Library:A_Single_Pad, F.Cu at (195.6, 185.4)
- added REF**: A_Single_Pad, Library:A_Single_Pad, F.Cu at (45.7, 152.4)
- added REF**: A_Single_Pad, Library:A_Single_Pad, F.Cu at (246.4, 182.9)
- added REF**: A_Single_Pad, Library:A_Single_Pad, F.Cu at (50.8, 175.3)
- added REF**: A_Single_Pad, Library:A_Single_Pad, F.Cu at (215.9, 182.9)
- added REF**: A_Single_Pad, Library:A_Single_Pad, F.Cu at (195.6, 190.5)
- added REF**: A_Single_Pad, Library:A_Single_Pad, F.Cu at (172.7, 61.0)
- added REF**: A_Single_Pad, Library:A_Single_Pad, F.Cu at (210.8, 190.5)
- added REF**: A_Single_Pad, Library:A_Single_Pad, F.Cu at (50.8, 167.6)
- added REF**: A_Single_Pad, Library:A_Single_Pad, F.Cu at (38.1, 154.9)
- added REF**: A_Single_Pad, Library:A_Single_Pad, F.Cu at (271.8, 172.7)
- added REF**: A_Single_Pad, Library:A_Single_Pad, F.Cu at (241.3, 170.2)
- added REF**: A_Single_Pad, Library:A_Single_Pad, F.Cu at (193.0, 193.0)
- added REF**: A_Single_Pad, Library:A_Single_Pad, F.Cu at (254.0, 165.1)
- added REF**: A_Single_Pad, Library:A_Single_Pad, F.Cu at (264.2, 167.6)
- added REF**: A_Single_Pad, Library:A_Single_Pad, F.Cu at (175.3, 73.7)
- added REF**: A_Single_Pad, Library:A_Single_Pad, F.Cu at (256.5, 177.8)
- added REF**: A_Single_Pad, Library:A_Single_Pad, F.Cu at (177.8, 61.0)
- added REF**: A_Single_Pad, Library:A_Single_Pad, F.Cu at (45.7, 160.0)
- added REF**: A_Single_Pad, Library:A_Single_Pad, F.Cu at (226.1, 188.0)
- added REF**: A_Single_Pad, Library:A_Single_Pad, F.Cu at (160.0, 76.2)
- added REF**: A_Single_Pad, Library:A_Single_Pad, F.Cu at (243.8, 188.0)
- added REF**: A_Single_Pad, Library:A_Single_Pad, F.Cu at (162.6, 61.0)
- added REF**: A_Single_Pad, Library:A_Single_Pad, F.Cu at (241.3, 167.6)
- added REF**: A_Single_Pad, Library:A_Single_Pad, F.Cu at (228.6, 188.0)
- added REF**: A_Single_Pad, Library:A_Single_Pad, F.Cu at (167.6, 63.5)
- added REF**: A_Single_Pad, Library:A_Single_Pad, F.Cu at (50.8, 170.2)
- added REF**: A_Single_Pad, Library:A_Single_Pad, F.Cu at (38.1, 170.2)
- added REF**: A_Single_Pad, Library:A_Single_Pad, F.Cu at (269.2, 177.8)
- added REF**: A_Single_Pad, Library:A_Single_Pad, F.Cu at (210.8, 188.0)
- added REF**: A_Single_Pad, Library:A_Single_Pad, F.Cu at (218.4, 188.0)
- added REF**: A_Single_Pad, Library:A_Single_Pad, F.Cu at (203.2, 185.4)
- added REF**: A_Single_Pad, Library:A_Single_Pad, F.Cu at (231.1, 190.5)
- added REF**: A_Single_Pad, Library:A_Single_Pad, F.Cu at (226.1, 190.5)
- added REF**: A_Single_Pad, Library:A_Single_Pad, F.Cu at (213.4, 190.5)
- added REF**: A_Single_Pad, Library:A_Single_Pad, F.Cu at (203.2, 190.5)
- added REF**: A_Single_Pad, Library:A_Single_Pad, F.Cu at (248.9, 172.7)
- added REF**: A_Single_Pad, Library:A_Single_Pad, F.Cu at (248.9, 193.0)
- added REF**: A_Single_Pad, Library:A_Single_Pad, F.Cu at (43.2, 162.6)
- added REF**: A_Single_Pad, Library:A_Single_Pad, F.Cu at (271.8, 165.1)
- added REF**: A_Single_Pad, Library:A_Single_Pad, F.Cu at (226.1, 193.0)
- added REF**: A_Single_Pad, Library:A_Single_Pad, F.Cu at (58.4, 152.4)
- added REF**: A_Single_Pad, Library:A_Single_Pad, F.Cu at (190.5, 188.0)
- added REF**: A_Single_Pad, Library:A_Single_Pad, F.Cu at (165.1, 50.8)
- added REF**: A_Single_Pad, Library:A_Single_Pad, F.Cu at (50.8, 152.4)
- added REF**: A_Single_Pad, Library:A_Single_Pad, F.Cu at (213.4, 185.4)
- added REF**: A_Single_Pad, Library:A_Single_Pad, F.Cu at (208.3, 193.0)
- added REF**: A_Single_Pad, Library:A_Single_Pad, F.Cu at (162.6, 71.1)
- added REF**: A_Single_Pad, Library:A_Single_Pad, F.Cu at (246.4, 167.6)
- added REF**: A_Single_Pad, Library:A_Single_Pad, F.Cu at (40.6, 157.5)
- added REF**: A_Single_Pad, Library:A_Single_Pad, F.Cu at (259.1, 175.3)
- added REF**: A_Single_Pad, Library:A_Single_Pad, F.Cu at (58.4, 149.9)
- added REF**: A_Single_Pad, Library:A_Single_Pad, F.Cu at (266.7, 180.3)
- added REF**: A_Single_Pad, Library:A_Single_Pad, F.Cu at (40.6, 182.9)
- added REF**: A_Single_Pad, Library:A_Single_Pad, F.Cu at (48.3, 162.6)
- added REF**: A_Single_Pad, Library:A_Single_Pad, F.Cu at (233.7, 185.4)
- added REF**: A_Single_Pad, Library:A_Single_Pad, F.Cu at (195.6, 188.0)
- added REF**: A_Single_Pad, Library:A_Single_Pad, F.Cu at (208.3, 188.0)
- added REF**: A_Single_Pad, Library:A_Single_Pad, F.Cu at (264.2, 162.6)
- added REF**: A_Single_Pad, Library:A_Single_Pad, F.Cu at (238.8, 175.3)
- added REF**: A_Single_Pad, Library:A_Single_Pad, F.Cu at (165.1, 66.0)
- added REF**: A_Single_Pad, Library:A_Single_Pad, F.Cu at (38.1, 160.0)
- added REF**: A_Single_Pad, Library:A_Single_Pad, F.Cu at (261.6, 165.1)
- added REF**: A_Single_Pad, Library:A_Single_Pad, F.Cu at (243.8, 175.3)
- added REF**: A_Single_Pad, Library:A_Single_Pad, F.Cu at (271.8, 162.6)
- added REF**: A_Single_Pad, Library:A_Single_Pad, F.Cu at (182.9, 73.7)
- added REF**: A_Single_Pad, Library:A_Single_Pad, F.Cu at (38.1, 165.1)
- added REF**: A_Single_Pad, Library:A_Single_Pad, F.Cu at (165.1, 68.6)
- added REF**: A_Single_Pad, Library:A_Single_Pad, F.Cu at (251.5, 193.0)
- added REF**: A_Single_Pad, Library:A_Single_Pad, F.Cu at (243.8, 162.6)
- added REF**: A_Single_Pad, Library:A_Single_Pad, F.Cu at (269.2, 162.6)
- added REF**: A_Single_Pad, Library:A_Single_Pad, F.Cu at (256.5, 165.1)
- added REF**: A_Single_Pad, Library:A_Single_Pad, F.Cu at (256.5, 175.3)
- added REF**: A_Single_Pad, Library:A_Single_Pad, F.Cu at (172.7, 66.0)
- added REF**: A_Single_Pad, Library:A_Single_Pad, F.Cu at (45.7, 182.9)
- added REF**: A_Single_Pad, Library:A_Single_Pad, F.Cu at (162.6, 63.5)
- added REF**: A_Single_Pad, Library:A_Single_Pad, F.Cu at (53.3, 152.4)
- added REF**: A_Single_Pad, Library:A_Single_Pad, F.Cu at (236.2, 193.0)
- added REF**: A_Single_Pad, Library:A_Single_Pad, F.Cu at (248.9, 188.0)
- added REF**: A_Single_Pad, Library:A_Single_Pad, F.Cu at (175.3, 53.3)
- added REF**: A_Single_Pad, Library:A_Single_Pad, F.Cu at (172.7, 71.1)
- added REF**: A_Single_Pad, Library:A_Single_Pad, F.Cu at (53.3, 180.3)
- added REF**: A_Single_Pad, Library:A_Single_Pad, F.Cu at (205.7, 185.4)
- added REF**: A_Single_Pad, Library:A_Single_Pad, F.Cu at (264.2, 193.0)
- added REF**: A_Single_Pad, Library:A_Single_Pad, F.Cu at (259.1, 180.3)
- added REF**: A_Single_Pad, Library:A_Single_Pad, F.Cu at (228.6, 185.4)
- added REF**: A_Single_Pad, Library:A_Single_Pad, F.Cu at (200.7, 190.5)
- added REF**: A_Single_Pad, Library:A_Single_Pad, F.Cu at (55.9, 172.7)
- added REF**: A_Single_Pad, Library:A_Single_Pad, F.Cu at (248.9, 167.6)
- added REF**: A_Single_Pad, Library:A_Single_Pad, F.Cu at (198.1, 190.5)
- added REF**: A_Single_Pad, Library:A_Single_Pad, F.Cu at (236.2, 188.0)
- added REF**: A_Single_Pad, Library:A_Single_Pad, F.Cu at (40.6, 175.3)
- added REF**: A_Single_Pad, Library:A_Single_Pad, F.Cu at (200.7, 188.0)
- added REF**: A_Single_Pad, Library:A_Single_Pad, F.Cu at (264.2, 185.4)
- added REF**: A_Single_Pad, Library:A_Single_Pad, F.Cu at (160.0, 71.1)
- added REF**: A_Single_Pad, Library:A_Single_Pad, F.Cu at (172.7, 55.9)
- added REF**: A_Single_Pad, Library:A_Single_Pad, F.Cu at (53.3, 175.3)
- added REF**: A_Single_Pad, Library:A_Single_Pad, F.Cu at (48.3, 177.8)
- added REF**: A_Single_Pad, Library:A_Single_Pad, F.Cu at (170.2, 76.2)
- added REF**: A_Single_Pad, Library:A_Single_Pad, F.Cu at (274.3, 170.2)
- added REF**: A_Single_Pad, Library:A_Single_Pad, F.Cu at (266.7, 172.7)
- added REF**: A_Single_Pad, Library:A_Single_Pad, F.Cu at (266.7, 167.6)
- added REF**: A_Single_Pad, Library:A_Single_Pad, F.Cu at (182.9, 71.1)
- added REF**: A_Single_Pad, Library:A_Single_Pad, F.Cu at (58.4, 154.9)
- added REF**: A_Single_Pad, Library:A_Single_Pad, F.Cu at (236.2, 162.6)
- added REF**: A_Single_Pad, Library:A_Single_Pad, F.Cu at (175.3, 58.4)
- added REF**: A_Single_Pad, Library:A_Single_Pad, F.Cu at (53.3, 154.9)
- added REF**: A_Single_Pad, Library:A_Single_Pad, F.Cu at (45.7, 172.7)
- added REF**: A_Single_Pad, Library:A_Single_Pad, F.Cu at (162.6, 68.6)
- added REF**: A_Single_Pad, Library:A_Single_Pad, F.Cu at (43.2, 160.0)
- added REF**: A_Single_Pad, Library:A_Single_Pad, F.Cu at (198.1, 193.0)
- added REF**: A_Single_Pad, Library:A_Single_Pad, F.Cu at (254.0, 167.6)
- added REF**: A_Single_Pad, Library:A_Single_Pad, F.Cu at (160.0, 61.0)
- added REF**: A_Single_Pad, Library:A_Single_Pad, F.Cu at (266.7, 182.9)
- added REF**: A_Single_Pad, Library:A_Single_Pad, F.Cu at (218.4, 190.5)
- added REF**: A_Single_Pad, Library:A_Single_Pad, F.Cu at (233.7, 188.0)
- added REF**: A_Single_Pad, Library:A_Single_Pad, F.Cu at (48.3, 154.9)
- added REF**: A_Single_Pad, Library:A_Single_Pad, F.Cu at (231.1, 182.9)
- added REF**: A_Single_Pad, Library:A_Single_Pad, F.Cu at (210.8, 185.4)
- added REF**: A_Single_Pad, Library:A_Single_Pad, F.Cu at (241.3, 162.6)
- added REF**: A_Single_Pad, Library:A_Single_Pad, F.Cu at (55.9, 149.9)
- added REF**: A_Single_Pad, Library:A_Single_Pad, F.Cu at (160.0, 50.8)
- added REF**: A_Single_Pad, Library:A_Single_Pad, F.Cu at (160.0, 55.9)
- added REF**: A_Single_Pad, Library:A_Single_Pad, F.Cu at (182.9, 55.9)
- added REF**: A_Single_Pad, Library:A_Single_Pad, F.Cu at (182.9, 76.2)
- added REF**: A_Single_Pad, Library:A_Single_Pad, F.Cu at (43.2, 170.2)
- added REF**: A_Single_Pad, Library:A_Single_Pad, F.Cu at (246.4, 165.1)
- added REF**: A_Single_Pad, Library:A_Single_Pad, F.Cu at (251.5, 177.8)
- added REF**: A_Single_Pad, Library:A_Single_Pad, F.Cu at (228.6, 190.5)
- added REF**: A_Single_Pad, Library:A_Single_Pad, F.Cu at (50.8, 160.0)
- added REF**: A_Single_Pad, Library:A_Single_Pad, F.Cu at (259.1, 177.8)
- added REF**: A_Single_Pad, Library:A_Single_Pad, F.Cu at (170.2, 71.1)
- added REF**: A_Single_Pad, Library:A_Single_Pad, F.Cu at (274.3, 177.8)
- added REF**: A_Single_Pad, Library:A_Single_Pad, F.Cu at (43.2, 149.9)
- added REF**: A_Single_Pad, Library:A_Single_Pad, F.Cu at (210.8, 182.9)
- added REF**: A_Single_Pad, Library:A_Single_Pad, F.Cu at (45.7, 180.3)
- added REF**: A_Single_Pad, Library:A_Single_Pad, F.Cu at (264.2, 188.0)
- added REF**: A_Single_Pad, Library:A_Single_Pad, F.Cu at (254.0, 188.0)
- added REF**: A_Single_Pad, Library:A_Single_Pad, F.Cu at (221.0, 188.0)
- added REF**: A_Single_Pad, Library:A_Single_Pad, F.Cu at (259.1, 182.9)
- added REF**: A_Single_Pad, Library:A_Single_Pad, F.Cu at (238.8, 180.3)
- added REF**: A_Single_Pad, Library:A_Single_Pad, F.Cu at (233.7, 172.7)
- added REF**: A_Single_Pad, Library:A_Single_Pad, F.Cu at (251.5, 167.6)
- added REF**: A_Single_Pad, Library:A_Single_Pad, F.Cu at (50.8, 154.9)
- added REF**: A_Single_Pad, Library:A_Single_Pad, F.Cu at (266.7, 177.8)
- added REF**: A_Single_Pad, Library:A_Single_Pad, F.Cu at (167.6, 66.0)
- added REF**: A_Single_Pad, Library:A_Single_Pad, F.Cu at (271.8, 167.6)
- added REF**: A_Single_Pad, Library:A_Single_Pad, F.Cu at (167.6, 71.1)
- added REF**: A_Single_Pad, Library:A_Single_Pad, F.Cu at (43.2, 154.9)
- added REF**: A_Single_Pad, Library:A_Single_Pad, F.Cu at (223.5, 193.0)
- added REF**: A_Single_Pad, Library:A_Single_Pad, F.Cu at (53.3, 182.9)
- added REF**: A_Single_Pad, Library:A_Single_Pad, F.Cu at (241.3, 182.9)
- added REF**: A_Single_Pad, Library:A_Single_Pad, F.Cu at (233.7, 165.1)
- added REF**: A_Single_Pad, Library:A_Single_Pad, F.Cu at (162.6, 76.2)
- added REF**: A_Single_Pad, Library:A_Single_Pad, F.Cu at (177.8, 68.6)
- added REF**: A_Single_Pad, Library:A_Single_Pad, F.Cu at (185.4, 73.7)
- added REF**: A_Single_Pad, Library:A_Single_Pad, F.Cu at (167.6, 53.3)
- added REF**: A_Single_Pad, Library:A_Single_Pad, F.Cu at (48.3, 157.5)
- added REF**: A_Single_Pad, Library:A_Single_Pad, F.Cu at (271.8, 182.9)
- added REF**: A_Single_Pad, Library:A_Single_Pad, F.Cu at (177.8, 76.2)
- added REF**: A_Single_Pad, Library:A_Single_Pad, F.Cu at (167.6, 58.4)
- added REF**: A_Single_Pad, Library:A_Single_Pad, F.Cu at (248.9, 162.6)
- added REF**: A_Single_Pad, Library:A_Single_Pad, F.Cu at (55.9, 182.9)
- added REF**: A_Single_Pad, Library:A_Single_Pad, F.Cu at (193.0, 185.4)
- added REF**: A_Single_Pad, Library:A_Single_Pad, F.Cu at (223.5, 188.0)
- added REF**: A_Single_Pad, Library:A_Single_Pad, F.Cu at (248.9, 177.8)
- added REF**: A_Single_Pad, Library:A_Single_Pad, F.Cu at (231.1, 193.0)
- added REF**: A_Single_Pad, Library:A_Single_Pad, F.Cu at (40.6, 160.0)
- added REF**: A_Single_Pad, Library:A_Single_Pad, F.Cu at (221.0, 190.5)
- added REF**: A_Single_Pad, Library:A_Single_Pad, F.Cu at (40.6, 165.1)
- added REF**: A_Single_Pad, Library:A_Single_Pad, F.Cu at (43.2, 157.5)
- added REF**: A_Single_Pad, Library:A_Single_Pad, F.Cu at (160.0, 58.4)
- added REF**: A_Single_Pad, Library:A_Single_Pad, F.Cu at (256.5, 182.9)
- added REF**: A_Single_Pad, Library:A_Single_Pad, F.Cu at (170.2, 58.4)
- added REF**: A_Single_Pad, Library:A_Single_Pad, F.Cu at (238.8, 193.0)
- added REF**: A_Single_Pad, Library:A_Single_Pad, F.Cu at (254.0, 193.0)
- added REF**: A_Single_Pad, Library:A_Single_Pad, F.Cu at (53.3, 149.9)
- added REF**: A_Single_Pad, Library:A_Single_Pad, F.Cu at (55.9, 154.9)
- added REF**: A_Single_Pad, Library:A_Single_Pad, F.Cu at (38.1, 167.6)
- added REF**: A_Single_Pad, Library:A_Single_Pad, F.Cu at (246.4, 172.7)
- added REF**: A_Single_Pad, Library:A_Single_Pad, F.Cu at (175.3, 68.6)
- added REF**: A_Single_Pad, Library:A_Single_Pad, F.Cu at (254.0, 162.6)
- added REF**: A_Single_Pad, Library:A_Single_Pad, F.Cu at (175.3, 50.8)
- added REF**: A_Single_Pad, Library:A_Single_Pad, F.Cu at (248.9, 180.3)
- added REF**: A_Single_Pad, Library:A_Single_Pad, F.Cu at (185.4, 76.2)
- added REF**: A_Single_Pad, Library:A_Single_Pad, F.Cu at (175.3, 55.9)
- added REF**: A_Single_Pad, Library:A_Single_Pad, F.Cu at (38.1, 177.8)
- added REF**: A_Single_Pad, Library:A_Single_Pad, F.Cu at (50.8, 172.7)
- added REF**: A_Single_Pad, Library:A_Single_Pad, F.Cu at (221.0, 193.0)
- added REF**: A_Single_Pad, Library:A_Single_Pad, F.Cu at (43.2, 167.6)
- added REF**: A_Single_Pad, Library:A_Single_Pad, F.Cu at (228.6, 193.0)
- added REF**: A_Single_Pad, Library:A_Single_Pad, F.Cu at (259.1, 188.0)
- added REF**: A_Single_Pad, Library:A_Single_Pad, F.Cu at (185.4, 68.6)
- added REF**: A_Single_Pad, Library:A_Single_Pad, F.Cu at (165.1, 76.2)
- added REF**: A_Single_Pad, Library:A_Single_Pad, F.Cu at (251.5, 170.2)
- added REF**: A_Single_Pad, Library:A_Single_Pad, F.Cu at (48.3, 182.9)
- added REF**: A_Single_Pad, Library:A_Single_Pad, F.Cu at (269.2, 182.9)
- added REF**: A_Single_Pad, Library:A_Single_Pad, F.Cu at (269.2, 172.7)
- added REF**: A_Single_Pad, Library:A_Single_Pad, F.Cu at (50.8, 180.3)
- added REF**: A_Single_Pad, Library:A_Single_Pad, F.Cu at (259.1, 165.1)
- added REF**: A_Single_Pad, Library:A_Single_Pad, F.Cu at (175.3, 63.5)
- added REF**: A_Single_Pad, Library:A_Single_Pad, F.Cu at (213.4, 188.0)
- added REF**: A_Single_Pad, Library:A_Single_Pad, F.Cu at (254.0, 190.5)
- added REF**: A_Single_Pad, Library:A_Single_Pad, F.Cu at (241.3, 193.0)
- added REF**: A_Single_Pad, Library:A_Single_Pad, F.Cu at (264.2, 175.3)
- added REF**: A_Single_Pad, Library:A_Single_Pad, F.Cu at (50.8, 157.5)
- added REF**: A_Single_Pad, Library:A_Single_Pad, F.Cu at (233.7, 193.0)
- added REF**: A_Single_Pad, Library:A_Single_Pad, F.Cu at (170.2, 66.0)
- added REF**: A_Single_Pad, Library:A_Single_Pad, F.Cu at (274.3, 167.6)
- added REF**: A_Single_Pad, Library:A_Single_Pad, F.Cu at (236.2, 190.5)
- added REF**: A_Single_Pad, Library:A_Single_Pad, F.Cu at (182.9, 66.0)
- added REF**: A_Single_Pad, Library:A_Single_Pad, F.Cu at (233.7, 162.6)
- added REF**: A_Single_Pad, Library:A_Single_Pad, F.Cu at (200.7, 185.4)
- added REF**: A_Single_Pad, Library:A_Single_Pad, F.Cu at (218.4, 193.0)
- added REF**: A_Single_Pad, Library:A_Single_Pad, F.Cu at (45.7, 149.9)
- added REF**: A_Single_Pad, Library:A_Single_Pad, F.Cu at (58.4, 157.5)
- added REF**: A_Single_Pad, Library:A_Single_Pad, F.Cu at (200.7, 193.0)
- added REF**: A_Single_Pad, Library:A_Single_Pad, F.Cu at (246.4, 185.4)
- added REF**: A_Single_Pad, Library:A_Single_Pad, F.Cu at (190.5, 182.9)
- added REF**: A_Single_Pad, Library:A_Single_Pad, F.Cu at (172.7, 76.2)
- added REF**: A_Single_Pad, Library:A_Single_Pad, F.Cu at (248.9, 175.3)
- added REF**: A_Single_Pad, Library:A_Single_Pad, F.Cu at (160.0, 73.7)
- added REF**: A_Single_Pad, Library:A_Single_Pad, F.Cu at (208.3, 182.9)
- added REF**: A_Single_Pad, Library:A_Single_Pad, F.Cu at (261.6, 182.9)
- added REF**: A_Single_Pad, Library:A_Single_Pad, F.Cu at (264.2, 180.3)
- added REF**: A_Single_Pad, Library:A_Single_Pad, F.Cu at (167.6, 76.2)
- added REF**: A_Single_Pad, Library:A_Single_Pad, F.Cu at (172.7, 68.6)
- added REF**: A_Single_Pad, Library:A_Single_Pad, F.Cu at (55.9, 165.1)
- added REF**: A_Single_Pad, Library:A_Single_Pad, F.Cu at (198.1, 185.4)
- added REF**: A_Single_Pad, Library:A_Single_Pad, F.Cu at (175.3, 71.1)
- added REF**: A_Single_Pad, Library:A_Single_Pad, F.Cu at (264.2, 172.7)
- added REF**: A_Single_Pad, Library:A_Single_Pad, F.Cu at (251.5, 190.5)
- added REF**: A_Single_Pad, Library:A_Single_Pad, F.Cu at (236.2, 177.8)
- added REF**: A_Single_Pad, Library:A_Single_Pad, F.Cu at (38.1, 162.6)
- added REF**: A_Single_Pad, Library:A_Single_Pad, F.Cu at (58.4, 165.1)
- added REF**: A_Single_Pad, Library:A_Single_Pad, F.Cu at (160.0, 63.5)
- added REF**: A_Single_Pad, Library:A_Single_Pad, F.Cu at (251.5, 165.1)
- added REF**: A_Single_Pad, Library:A_Single_Pad, F.Cu at (170.2, 53.3)
- added REF**: A_Single_Pad, Library:A_Single_Pad, F.Cu at (45.7, 175.3)
- added REF**: A_Single_Pad, Library:A_Single_Pad, F.Cu at (165.1, 55.9)
- added REF**: A_Single_Pad, Library:A_Single_Pad, F.Cu at (233.7, 175.3)
- added REF**: A_Single_Pad, Library:A_Single_Pad, F.Cu at (190.5, 193.0)
- added REF**: A_Single_Pad, Library:A_Single_Pad, F.Cu at (254.0, 182.9)
- added REF**: A_Single_Pad, Library:A_Single_Pad, F.Cu at (256.5, 170.2)
- added REF**: A_Single_Pad, Library:A_Single_Pad, F.Cu at (177.8, 63.5)
- added REF**: A_Single_Pad, Library:A_Single_Pad, F.Cu at (261.6, 190.5)
- added REF**: A_Single_Pad, Library:A_Single_Pad, F.Cu at (241.3, 172.7)
- added REF**: A_Single_Pad, Library:A_Single_Pad, F.Cu at (165.1, 53.3)
- added REF**: A_Single_Pad, Library:A_Single_Pad, F.Cu at (243.8, 167.6)
- added REF**: A_Single_Pad, Library:A_Single_Pad, F.Cu at (233.7, 182.9)
- added REF**: A_Single_Pad, Library:A_Single_Pad, F.Cu at (264.2, 190.5)
- added REF**: A_Single_Pad, Library:A_Single_Pad, F.Cu at (254.0, 177.8)
- added REF**: A_Single_Pad, Library:A_Single_Pad, F.Cu at (233.7, 180.3)
- added REF**: A_Single_Pad, Library:A_Single_Pad, F.Cu at (271.8, 170.2)
- added REF**: A_Single_Pad, Library:A_Single_Pad, F.Cu at (177.8, 53.3)
- added REF**: A_Single_Pad, Library:A_Single_Pad, F.Cu at (182.9, 53.3)
- added REF**: A_Single_Pad, Library:A_Single_Pad, F.Cu at (43.2, 180.3)
- added REF**: A_Single_Pad, Library:A_Single_Pad, F.Cu at (261.6, 180.3)
- added REF**: A_Single_Pad, Library:A_Single_Pad, F.Cu at (246.4, 170.2)
- added REF**: A_Single_Pad, Library:A_Single_Pad, F.Cu at (180.3, 50.8)
- added REF**: A_Single_Pad, Library:A_Single_Pad, F.Cu at (53.3, 157.5)
- added REF**: A_Single_Pad, Library:A_Single_Pad, F.Cu at (58.4, 170.2)
- added REF**: A_Single_Pad, Library:A_Single_Pad, F.Cu at (43.2, 172.7)
- added REF**: A_Single_Pad, Library:A_Single_Pad, F.Cu at (236.2, 180.3)
- added REF**: A_Single_Pad, Library:A_Single_Pad, F.Cu at (248.9, 170.2)
- added REF**: A_Single_Pad, Library:A_Single_Pad, F.Cu at (48.3, 170.2)
- added REF**: A_Single_Pad, Library:A_Single_Pad, F.Cu at (261.6, 177.8)
- added REF**: A_Single_Pad, Library:A_Single_Pad, F.Cu at (185.4, 58.4)
- added REF**: A_Single_Pad, Library:A_Single_Pad, F.Cu at (246.4, 193.0)
- added REF**: A_Single_Pad, Library:A_Single_Pad, F.Cu at (261.6, 172.7)
- added REF**: A_Single_Pad, Library:A_Single_Pad, F.Cu at (205.7, 190.5)
- added REF**: A_Single_Pad, Library:A_Single_Pad, F.Cu at (238.8, 177.8)
- added REF**: A_Single_Pad, Library:A_Single_Pad, F.Cu at (243.8, 170.2)
- added REF**: A_Single_Pad, Library:A_Single_Pad, F.Cu at (58.4, 182.9)
- added REF**: A_Single_Pad, Library:A_Single_Pad, F.Cu at (231.1, 188.0)
- added REF**: A_Single_Pad, Library:A_Single_Pad, F.Cu at (274.3, 162.6)
- added REF**: A_Single_Pad, Library:A_Single_Pad, F.Cu at (261.6, 162.6)
- added REF**: A_Single_Pad, Library:A_Single_Pad, F.Cu at (48.3, 180.3)
- added REF**: A_Single_Pad, Library:A_Single_Pad, F.Cu at (243.8, 193.0)
- added REF**: A_Single_Pad, Library:A_Single_Pad, F.Cu at (55.9, 175.3)
- added REF**: A_Single_Pad, Library:A_Single_Pad, F.Cu at (48.3, 152.4)
- added REF**: A_Single_Pad, Library:A_Single_Pad, F.Cu at (170.2, 55.9)
- added REF**: A_Single_Pad, Library:A_Single_Pad, F.Cu at (48.3, 167.6)
- added REF**: A_Single_Pad, Library:A_Single_Pad, F.Cu at (205.7, 188.0)
- added REF**: A_Single_Pad, Library:A_Single_Pad, F.Cu at (256.5, 188.0)
- added REF**: A_Single_Pad, Library:A_Single_Pad, F.Cu at (203.2, 182.9)
- added REF**: A_Single_Pad, Library:A_Single_Pad, F.Cu at (175.3, 76.2)
- added REF**: A_Single_Pad, Library:A_Single_Pad, F.Cu at (160.0, 68.6)
- added REF**: A_Single_Pad, Library:A_Single_Pad, F.Cu at (238.8, 162.6)
- added REF**: A_Single_Pad, Library:A_Single_Pad, F.Cu at (182.9, 61.0)
- added REF**: A_Single_Pad, Library:A_Single_Pad, F.Cu at (238.8, 167.6)
- added REF**: A_Single_Pad, Library:A_Single_Pad, F.Cu at (172.7, 63.5)
- added REF**: A_Single_Pad, Library:A_Single_Pad, F.Cu at (50.8, 177.8)
- added REF**: A_Single_Pad, Library:A_Single_Pad, F.Cu at (256.5, 190.5)
- added REF**: A_Single_Pad, Library:A_Single_Pad, F.Cu at (165.1, 71.1)
- added REF**: A_Single_Pad, Library:A_Single_Pad, F.Cu at (167.6, 61.0)
- added REF**: A_Single_Pad, Library:A_Single_Pad, F.Cu at (167.6, 68.6)
- added REF**: A_Single_Pad, Library:A_Single_Pad, F.Cu at (233.7, 190.5)
- added REF**: A_Single_Pad, Library:A_Single_Pad, F.Cu at (243.8, 190.5)
- added REF**: A_Single_Pad, Library:A_Single_Pad, F.Cu at (269.2, 180.3)
- added REF**: A_Single_Pad, Library:A_Single_Pad, F.Cu at (55.9, 180.3)
- added REF**: A_Single_Pad, Library:A_Single_Pad, F.Cu at (238.8, 188.0)
- added REF**: A_Single_Pad, Library:A_Single_Pad, F.Cu at (38.1, 152.4)
- added REF**: A_Single_Pad, Library:A_Single_Pad, F.Cu at (180.3, 76.2)
- added REF**: A_Single_Pad, Library:A_Single_Pad, F.Cu at (223.5, 190.5)
- added REF**: A_Single_Pad, Library:A_Single_Pad, F.Cu at (274.3, 172.7)
- added REF**: A_Single_Pad, Library:A_Single_Pad, F.Cu at (58.4, 177.8)
- added REF**: A_Single_Pad, Library:A_Single_Pad, F.Cu at (50.8, 149.9)
- added REF**: A_Single_Pad, Library:A_Single_Pad, F.Cu at (175.3, 66.0)
- added REF**: A_Single_Pad, Library:A_Single_Pad, F.Cu at (182.9, 63.5)
- added REF**: A_Single_Pad, Library:A_Single_Pad, F.Cu at (160.0, 53.3)
- added REF**: A_Single_Pad, Library:A_Single_Pad, F.Cu at (208.3, 185.4)
- added REF**: A_Single_Pad, Library:A_Single_Pad, F.Cu at (40.6, 180.3)
- added REF**: A_Single_Pad, Library:A_Single_Pad, F.Cu at (233.7, 177.8)
- added REF**: A_Single_Pad, Library:A_Single_Pad, F.Cu at (246.4, 162.6)
- added REF**: A_Single_Pad, Library:A_Single_Pad, F.Cu at (248.9, 185.4)
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Connections:
- U2 pad 1: /HEC_Memory/RAM_A18 -> /HEC_IO/A7
- U2 pad 10: /HEC_IO/A2 -> /HEC_Memory/RAM_A13
- U2 pad 11: /HEC_IO/A1 -> /HEC_Memory/RAM_A14
- U2 pad 12: /HEC_IO/A0 -> /HEC_Memory/RAM_A15
- U2 pad 13: /HEC_IO/D0 -> /HEC_IO/D1
- U2 pad 14: /HEC_IO/D1 -> /HEC_IO/D3
- U2 pad 15: /HEC_IO/D2 -> /HEC_IO/D5
- U2 pad 19: /HEC_IO/D5 -> /HEC_IO/D4
- U2 pad 2: /HEC_Memory/RAM_A16 -> /HEC_IO/A6
- U2 pad 20: /HEC_IO/D4 -> /HEC_IO/D2
- U2 pad 21: /HEC_IO/D3 -> /HEC_IO/D0
- U2 pad 23: /HEC_Memory/RAM_A10 -> /HEC_Memory/RAM_A18
- U2 pad 25: /HEC_Memory/RAM_A11 -> /HEC_Memory/RAM_A17
- U2 pad 26: /HEC_Memory/RAM_A9 -> /HEC_Memory/RAM_A16
- U2 pad 27: /HEC_Memory/RAM_A8 -> /HEC_IO/A0
- U2 pad 28: /HEC_Memory/RAM_A13 -> /HEC_IO/A1
- U2 pad 3: /HEC_Memory/RAM_A14 -> /HEC_IO/A4
- U2 pad 30: /HEC_Memory/RAM_A17 -> /HEC_IO/A3
- U2 pad 31: /HEC_Memory/RAM_A15 -> /HEC_IO/A5
- U2 pad 4: /HEC_Memory/RAM_A12 -> /HEC_IO/A2
- U2 pad 5: /HEC_IO/A7 -> /HEC_Memory/RAM_A8
- U2 pad 6: /HEC_IO/A6 -> /HEC_Memory/RAM_A9
- U2 pad 7: /HEC_IO/A5 -> /HEC_Memory/RAM_A10
- U2 pad 8: /HEC_IO/A4 -> /HEC_Memory/RAM_A11
- U2 pad 9: /HEC_IO/A3 -> /HEC_Memory/RAM_A12
- U3 pad 1: /HEC_Memory/RAM_A18 -> /HEC_IO/A7
- U3 pad 10: /HEC_IO/A2 -> /HEC_Memory/RAM_A13
- U3 pad 11: /HEC_IO/A1 -> /HEC_Memory/RAM_A14
- U3 pad 12: /HEC_IO/A0 -> /HEC_Memory/RAM_A15
- U3 pad 13: /HEC_IO/D0 -> /HEC_IO/D1
- U3 pad 14: /HEC_IO/D1 -> /HEC_IO/D3
- U3 pad 15: /HEC_IO/D2 -> /HEC_IO/D5
- U3 pad 19: /HEC_IO/D5 -> /HEC_IO/D4
- U3 pad 2: /HEC_Memory/RAM_A16 -> /HEC_IO/A6
- U3 pad 20: /HEC_IO/D4 -> /HEC_IO/D2
- U3 pad 21: /HEC_IO/D3 -> /HEC_IO/D0
- U3 pad 23: /HEC_Memory/RAM_A10 -> /HEC_Memory/RAM_A18
- U3 pad 25: /HEC_Memory/RAM_A11 -> /HEC_Memory/RAM_A17
- U3 pad 26: /HEC_Memory/RAM_A9 -> /HEC_Memory/RAM_A16
- U3 pad 27: /HEC_Memory/RAM_A8 -> /HEC_IO/A0
- U3 pad 28: /HEC_Memory/RAM_A13 -> /HEC_IO/A1
- U3 pad 3: /HEC_Memory/RAM_A14 -> /HEC_IO/A4
- U3 pad 30: /HEC_Memory/RAM_A17 -> /HEC_IO/A3
- U3 pad 31: /HEC_Memory/RAM_A15 -> /HEC_IO/A5
- U3 pad 4: /HEC_Memory/RAM_A12 -> /HEC_IO/A2
- U3 pad 5: /HEC_IO/A7 -> /HEC_Memory/RAM_A8
- U3 pad 6: /HEC_IO/A6 -> /HEC_Memory/RAM_A9
- U3 pad 7: /HEC_IO/A5 -> /HEC_Memory/RAM_A10
- U3 pad 8: /HEC_IO/A4 -> /HEC_Memory/RAM_A11
- U3 pad 9: /HEC_IO/A3 -> /HEC_Memory/RAM_A12
- U5 pad 11: /HEC_Memory/RAM_A16 -> /HEC_Memory/ATTR_WI
- U5 pad 12: /HEC_Memory/RAM_A17 -> /HEC_Memory/ATTR_NX
- U5 pad 13: /HEC_Memory/RAM_A18 -> /HEC_Memory/ATTR_RI
- U5 pad 15: /HEC_Memory/RAM_A19 -> /HEC_Memory/ATTR_WP
- U5 pad 16: /HEC_Memory/ATTR_RI -> /HEC_Memory/RAM_A18
- U5 pad 17: /HEC_Memory/ATTR_NX -> /HEC_Memory/RAM_A17
- U5 pad 18: /HEC_Memory/ATTR_WI -> /HEC_Memory/RAM_A16
- U5 pad 19: /HEC_Memory/ATTR_WP -> /HEC_Memory/RAM_A19
Routing:
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
Commit message: Some routing attempt
Attempted to route some traces. 2-layer PCB seems to be achievable. It might just be a fool's arrogance.
Parts:
- moved C8 243.8 mm to (170.2, 45.7)
- moved C13 212.1 mm to (248.9, 88.9), turned to 90 degrees
- moved C14 191.9 mm to (208.3, 86.4)
- moved C12 101.7 mm to (180.3, 245.1)
- moved C16 91.0 mm to (63.5, 172.7)
- moved C15 52.9 mm to (155.0, 242.6)
- moved BUS1 20.3 mm to (116.8, 83.8)
- moved BUS2 20.3 mm to (96.5, 83.8)
Routing:
- net L: track 203.2 -> 423.1 mm
- net H: track 132.1 -> 303.2 mm
- net Net-(U36-Q4): track 0.00 -> 79.4 mm, vias 0 -> 1
- net Net-(U36-Q7): track 0.00 -> 67.0 mm, vias 0 -> 1
- net Net-(J8-D3): track 0.00 -> 62.0 mm, vias 0 -> 1
- net /HEC_IO/AUDIO_R: track 64.1 -> 126.0 mm
- net Net-(U36-Q6): track 0.00 -> 59.6 mm, vias 0 -> 1
- net Net-(U36-Q5): track 0.00 -> 59.6 mm, vias 0 -> 1
- net Net-(U43-P22/MSDO): track 0.00 -> 58.3 mm
- net Net-(J8-D4): track 0.00 -> 53.4 mm, vias 0 -> 1
- net Net-(U43-P23/MSCO): track 0.00 -> 52.2 mm
- net /HEC_IO/AUDIO_L: track 64.1 -> 116.1 mm
- net Net-(J8-DATA): track 0.00 -> 49.3 mm, vias 0 -> 1
- net Net-(RN5-R4): track 0.00 -> 43.8 mm
- net Net-(RN5-R2): track 0.00 -> 35.9 mm, vias 0 -> 1
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